Commit message: Documentation and cleanup of initial commit for sub simulation

File: simulation/mantaray_description/urdf/gazebo.xacro (robot description, xacro)
@@ -2,11 +2,11 @@
 <robot xmlns:xacro="http://www.ros.org/wiki/xacro">
     <!-- Center of buoyancy -->
-    <xacro:property name="mantaray_cob" value="0 0 0"/>
+    <xacro:property name="mantaray_cob" value="0 0 0"/> <!-- Random value -->
     <!-- Vehicle's actual volume (Gazebo cannot compute the volume out of the mesh) -->
     <xacro:property name="mantaray_volume" value="1.83826"/> <!-- Taken from RexRov2-->
     <!-- Describing the dimensions of the vehicle's bounding box -->
-    <xacro:property name="mantaray_length" value="2.6"/><!-- Taken from RexRov2-->
-    <xacro:property name="mantaray_width"  value="1.5"/><!-- Taken from RexRov2-->
-    <xacro:property name="mantaray_height" value="1.6"/><!-- Taken from RexRov2-->
+    <xacro:property name="mantaray_length" value="0.629158"/> <!-- Might have mixed up length and width-->
+    <xacro:property name="mantaray_width"  value="0.80518"/>
+    <xacro:property name="mantaray_height" value="0.33782"/>
     <xacro:macro name="mantaray_hydro_model" params="namespace">
       <!-- List of hydrodynamic models this robot's links -->
