Commit message: Made the propeller into the T-200 one

File: simulation/mantaray_description/urdf/snippets.xacro (robot description, xacro)
@@ -7,5 +7,6 @@
   over propeller's frame X-axis in DAE (Collada) or STL format.
   -->
-  <xacro:property name="prop_mesh_file" value="file://$(find mantaray_description)/meshes/Propeller.dae"/>
+  <!-- I stole this dae file from https://github.com/francisc0garcia/robdos_sim/blob/master/models/robdos_model_thrust.dae -->
+  <xacro:property name="prop_mesh_file" value="file://$(find mantaray_description)/meshes/robdos_model_thrust.dae"/>
   <!--
     Thruster macro with integration of joint and link. The thrusters should
@@ -17,5 +18,5 @@
       namespace="${namespace}"
       thruster_id="${thruster_id}"
-      mesh_filename="file://$(find mantaray_description)/meshes/Propeller.dae"
+      mesh_filename="file://$(find mantaray_description)/meshes/robdos_model_thrust.dae"
       dyn_time_constant="0.05"
       rotor_constant="0.026546960744430276">

Commit message: The actuator configuration that I was previously using wasn't working. This one does and it moves the thrusters properly.

File: simulation/mantaray_description/urdf/snippets.xacro (robot description, xacro)
@@ -13,5 +13,5 @@
     be initialized in the actuators.xacro file.
   -->
-  <xacro:macro name="thruster_macro" params="namespace thruster_id *origin">
+  <!-- <xacro:macro name="thruster_macro" params="namespace thruster_id *origin">
     <joint name="${namespace}/thruster_${thruster_id}_joint" type="continuous">
       <xacro:insert_block name="origin"/>
@@ -53,6 +53,6 @@
       </plugin>
     </gazebo>
-  </xacro:macro>
-  <!-- <xacro:macro name="thruster_macro"
+  </xacro:macro> -->
+  <xacro:macro name="thruster_macro"
     params="namespace thruster_id *origin">
     <xacro:thruster_module_first_order_basic_fcn_macro
@@ -64,5 +64,5 @@
       <xacro:insert_block name="origin"/>
     </xacro:thruster_module_first_order_basic_fcn_macro>
-  </xacro:macro> -->
+  </xacro:macro>
   <!-- Ask david about dynaic time constant -->
   <!-- Look at the datasheet for rotor constant -->
