Commit message: Adjusting thrusters on the model. Trying to get them to move the sub correctly.

File: simulation/mantaray_description/urdf/actuators.xacro (robot description, xacro)
@@ -10,20 +10,26 @@
     <!-- Taken from RexRov2-->
     <xacro:thruster_macro namespace="${namespace}" thruster_id="0"> <!-- I inputed-->
-      <origin xyz="0.25518 -0.337990 0.211387" rpy="0 0 ${90*d2r}"/>
+      <origin xyz="-0.27 -0.294170 0.244899" rpy="0 0 ${90*d2r}"/>
     </xacro:thruster_macro>
-    <!-- <xacro:thruster_macro namespace="${namespace}" thruster_id="1">
-      <origin xyz="-0.8217 0 0.589" rpy="0 ${-75*d2r} 0"/>
+    <xacro:thruster_macro namespace="${namespace}" thruster_id="1">
+      <origin xyz="0.27 -0.294170 0.244899" rpy="0 0 ${90*d2r}"/>
     </xacro:thruster_macro>
     <xacro:thruster_macro namespace="${namespace}" thruster_id="2">
-      <origin xyz="0.8654 -0.5322 0.5332" rpy="0 ${-67.5*d2r} ${90*d2r}"/>
+      <origin xyz="0.27 0.294170 0.244899" rpy="0 ${90*d2r} 0"/>
     </xacro:thruster_macro>
-    <xacro:thruster_macro namespace="${namespace}" thruster_id="3">
-      <origin xyz="0.8654 0.5322 0.5332" rpy="0 ${67.5*d2r} ${90*d2r}"/>
+    <!-- <xacro:thruster_macro namespace="${namespace}" thruster_id="3">
+      <origin xyz="0.298572 0.356203 0.244899" rpy="0 ${67.5*d2r} ${90*d2r}"/>
     </xacro:thruster_macro>
     <xacro:thruster_macro namespace="${namespace}" thruster_id="4">
-      <origin xyz="-0.7076 0.5129 0.2404" rpy="0 0 ${25*d2r}"/>
+      <origin xyz="0.270130 0.164922 0.145563" rpy="0 0 ${25*d2r}"/>
     </xacro:thruster_macro>
     <xacro:thruster_macro namespace="${namespace}" thruster_id="5">
-      <origin xyz="-0.7076 -0.5129 0.2404" rpy="0 0 ${-25*d2r}"/>
+      <origin xyz="-0.193622 0.207182 0.145563" rpy="0 0 ${-25*d2r}"/>
+    </xacro:thruster_macro>
+    <xacro:thruster_macro namespace="${namespace}" thruster_id="6">
+      <origin xyz="-0.281372 -0.150723 0.145563" rpy="0 0 ${-25*d2r}"/>
+    </xacro:thruster_macro>
+    <xacro:thruster_macro namespace="${namespace}" thruster_id="7">
+      <origin xyz="0.193622 -0.200534 0.145563" rpy="0 0 ${-25*d2r}"/>
     </xacro:thruster_macro> -->
     <!-- Instantiate fins, if necessary -->

File: simulation/mantaray_description/urdf/snippets.xacro (robot description, xacro)
@@ -13,5 +13,46 @@
     be initialized in the actuators.xacro file.
   -->
-  <xacro:macro name="thruster_macro"
+  <xacro:macro name="thruster_macro" params="namespace thruster_id *origin">
+    <joint name="${namespace}/thruster_${thruster_id}_joint" type="continuous">
+      <xacro:insert_block name="origin"/>
+      <axis xyz="0 0 1"/>
+      <parent link="${namespace}/base_link"/>
+      <child link="${namespace}/thruster_${thruster_id}"/>
+    </joint>
+    <link name="${namespace}/thruster_${thruster_id}">
+      <xacro:box_inertial x="0" y="0" z="0" mass="0.001">
+        <origin xyz="0 0 0" rpy="0 0 0"/>
+      </xacro:box_inertial>
+      <visual>
+        <origin rpy="0 0 0" xyz="0 0 0"/>
+        <geometry>
+          <mesh filename="${prop_mesh_file}" scale="1.7 1.7 1.7"/>
+        </geometry>
+      </visual>
+      <collision>
+        <geometry>
+          <cylinder length="0.000001" radius="0.000001"/>
+        </geometry>
+        <origin xyz="0 0 0" rpy="0 ${0.5*pi} 0"/>
+      </collision>
+    </link>
+    <gazebo>
+      <plugin name="${namespace}_${thruster_id}_thruster_model" filename="libuuv_thruster_ros_plugin.so">
+        <linkName>${namespace}/thruster_${thruster_id}</linkName>
+        <jointName>${namespace}/thruster_${thruster_id}_joint</jointName>
+        <thrustTopic>${namespace}/thrusters/${thruster_id}/thrust</thrustTopic>
+        <inputTopic>${namespace}/thrusters/${thruster_id}/input</inputTopic>
+        <dynamics>
+          <type>FirstOrder</type>
+          <timeConstant>0.05</timeConstant>
+        </dynamics>
+        <conversion>
+          <type>Basic</type>
+          <rotorConstant>0.00031</rotorConstant>
+        </conversion>
+      </plugin>
+    </gazebo>
+  </xacro:macro>
+  <!-- <xacro:macro name="thruster_macro"
     params="namespace thruster_id *origin">
     <xacro:thruster_module_first_order_basic_fcn_macro
@@ -23,5 +64,5 @@
       <xacro:insert_block name="origin"/>
     </xacro:thruster_module_first_order_basic_fcn_macro>
-  </xacro:macro>
+  </xacro:macro> -->
   <!-- Ask david about dynaic time constant -->
   <!-- Look at the datasheet for rotor constant -->

Commit message: Tried to get the thrusters aligned and fix their rotation when actuated - Billy and William

File: simulation/mantaray_description/urdf/actuators.xacro (robot description, xacro)
@@ -13,16 +13,20 @@
     </xacro:thruster_macro>
     <xacro:thruster_macro namespace="${namespace}" thruster_id="1">
-      <origin xyz="0.27 -0.294170 0.244899" rpy="0 0 ${90*d2r}"/>
+      <origin xyz="0.27 -0.384170 0.244899" rpy="0 0 ${270*d2r}"/>
     </xacro:thruster_macro>
+                                    <!-- 0.238 -0.294170 0.244899 -->
     <xacro:thruster_macro namespace="${namespace}" thruster_id="2">
-      <origin xyz="0.27 0.294170 0.244899" rpy="0 ${90*d2r} 0"/>
+      <origin xyz="0.27 0.294170 0.244899" rpy="0 0 ${270*d2r}"/>
     </xacro:thruster_macro>
-    <!-- <xacro:thruster_macro namespace="${namespace}" thruster_id="3">
-      <origin xyz="0.298572 0.356203 0.244899" rpy="0 ${67.5*d2r} ${90*d2r}"/>
+    <xacro:thruster_macro namespace="${namespace}" thruster_id="3">
+      <origin xyz="-0.27 0.384170 0.244899" rpy="0 0 ${90*d2r}"/>
     </xacro:thruster_macro>
     <xacro:thruster_macro namespace="${namespace}" thruster_id="4">
-      <origin xyz="0.270130 0.164922 0.145563" rpy="0 0 ${25*d2r}"/>
+      <origin xyz="0.298572 0.356203 0.244899" rpy="${90*d2r} 0 0"/>
     </xacro:thruster_macro>
     <xacro:thruster_macro namespace="${namespace}" thruster_id="5">
+      <origin xyz="0.270130 0.164922 0.244899" rpy="0 ${90*d2r} 0"/>
+    </xacro:thruster_macro>
+    <!-- <xacro:thruster_macro namespace="${namespace}" thruster_id="5">
       <origin xyz="-0.193622 0.207182 0.145563" rpy="0 0 ${-25*d2r}"/>
     </xacro:thruster_macro>

Commit message: Got the thrusters to rotate properly and currently adding all the thrusters to their correct positions

File: simulation/mantaray_description/urdf/actuators.xacro (robot description, xacro)
@@ -10,21 +10,21 @@
     <!-- Taken from RexRov2-->
     <xacro:thruster_macro namespace="${namespace}" thruster_id="0"> <!-- I inputed-->
-      <origin xyz="-0.27 -0.294170 0.244899" rpy="0 0 ${90*d2r}"/>
+      <origin xyz="-0.25 -0.34 0.244899" rpy="0 ${90*d2r} 0"/>
     </xacro:thruster_macro>
     <xacro:thruster_macro namespace="${namespace}" thruster_id="1">
-      <origin xyz="0.27 -0.384170 0.244899" rpy="0 0 ${270*d2r}"/>
+      <origin xyz="0.25 -0.34 0.244899" rpy="0 ${90*d2r} 0"/>
     </xacro:thruster_macro>
                                     <!-- 0.238 -0.294170 0.244899 -->
     <xacro:thruster_macro namespace="${namespace}" thruster_id="2">
-      <origin xyz="0.27 0.294170 0.244899" rpy="0 0 ${270*d2r}"/>
+      <origin xyz="0.25 0.34 0.244899" rpy="0 ${90*d2r} 0"/>
     </xacro:thruster_macro>
     <xacro:thruster_macro namespace="${namespace}" thruster_id="3">
-      <origin xyz="-0.27 0.384170 0.244899" rpy="0 0 ${90*d2r}"/>
+      <origin xyz="-0.25 0.34 0.244899" rpy="0 ${90*d2r} 0"/>
     </xacro:thruster_macro>
     <xacro:thruster_macro namespace="${namespace}" thruster_id="4">
-      <origin xyz="0.298572 0.356203 0.244899" rpy="${90*d2r} 0 0"/>
+      <origin xyz="-0.25 0.15 0.244899" rpy="${90*d2r} 0 ${30*d2r}"/>
     </xacro:thruster_macro>
     <xacro:thruster_macro namespace="${namespace}" thruster_id="5">
-      <origin xyz="0.270130 0.164922 0.244899" rpy="0 ${90*d2r} 0"/>
+      <origin xyz="0.25 0.15 0.244899" rpy="${90*d2r} 0 ${330*d2r}"/>
     </xacro:thruster_macro>
     <!-- <xacro:thruster_macro namespace="${namespace}" thruster_id="5">

File: simulation/mantaray_description/urdf/snippets.xacro (robot description, xacro)
@@ -8,13 +8,13 @@
   -->
   <!-- I stole this dae file from https://github.com/francisc0garcia/robdos_sim/blob/master/models/robdos_model_thrust.dae -->
-  <xacro:property name="prop_mesh_file" value="file://$(find mantaray_description)/meshes/robdos_model_thrust.dae"/>
+  <xacro:property name="prop_mesh_file" value="file://$(find mantaray_description)/meshes/mantaray_prop.dae"/>
   <!--
     Thruster macro with integration of joint and link. The thrusters should
     be initialized in the actuators.xacro file.
   -->
-  <!-- <xacro:macro name="thruster_macro" params="namespace thruster_id *origin">
+  <xacro:macro name="thruster_macro" params="namespace thruster_id *origin">
     <joint name="${namespace}/thruster_${thruster_id}_joint" type="continuous">
       <xacro:insert_block name="origin"/>
-      <axis xyz="0 0 1"/>
+      <axis xyz="1 0 0"/>
       <parent link="${namespace}/base_link"/>
       <child link="${namespace}/thruster_${thruster_id}"/>
@@ -27,5 +27,5 @@
         <origin rpy="0 0 0" xyz="0 0 0"/>
         <geometry>
-          <mesh filename="${prop_mesh_file}" scale="1.7 1.7 1.7"/>
+          <mesh filename="${prop_mesh_file}" scale="1 1 1"/>
         </geometry>
       </visual>
@@ -34,5 +34,5 @@
           <cylinder length="0.000001" radius="0.000001"/>
         </geometry>
-        <origin xyz="0 0 0" rpy="0 ${0.5*pi} 0"/>
+        <origin xyz="0 0 0" rpy="0 0 0"/>
       </collision>
     </link>
@@ -41,6 +41,5 @@
         <linkName>${namespace}/thruster_${thruster_id}</linkName>
         <jointName>${namespace}/thruster_${thruster_id}_joint</jointName>
-        <thrustTopic>${namespace}/thrusters/${thruster_id}/thrust</thrustTopic>
-        <inputTopic>${namespace}/thrusters/${thruster_id}/input</inputTopic>
+        <thrusterID>${thruster_id}</thrusterID>
         <dynamics>
           <type>FirstOrder</type>
@@ -53,6 +52,9 @@
       </plugin>
     </gazebo>
-  </xacro:macro> -->
-  <xacro:macro name="thruster_macro"
+    <gazebo reference="${namespace}/thruster_${thruster_id}">
+      <selfCollide>false</selfCollide>
+    </gazebo>
+  </xacro:macro>
+  <!-- <xacro:macro name="thruster_macro"
     params="namespace thruster_id *origin">
     <xacro:thruster_module_first_order_basic_fcn_macro
@@ -64,5 +66,5 @@
       <xacro:insert_block name="origin"/>
     </xacro:thruster_module_first_order_basic_fcn_macro>
-  </xacro:macro>
+  </xacro:macro> -->
   <!-- Ask david about dynaic time constant -->
   <!-- Look at the datasheet for rotor constant -->

Commit message: Put thrusters in place

File: simulation/mantaray_description/urdf/actuators.xacro (robot description, xacro)
@@ -23,18 +23,15 @@
     </xacro:thruster_macro>
     <xacro:thruster_macro namespace="${namespace}" thruster_id="4">
-      <origin xyz="-0.25 0.15 0.244899" rpy="${90*d2r} 0 ${30*d2r}"/>
+      <origin xyz="-0.222 0.155 0.109" rpy="${90*d2r} 0 ${300*d2r}"/>
     </xacro:thruster_macro>
     <xacro:thruster_macro namespace="${namespace}" thruster_id="5">
-      <origin xyz="0.25 0.15 0.244899" rpy="${90*d2r} 0 ${330*d2r}"/>
-    </xacro:thruster_macro>
-    <!-- <xacro:thruster_macro namespace="${namespace}" thruster_id="5">
-      <origin xyz="-0.193622 0.207182 0.145563" rpy="0 0 ${-25*d2r}"/>
+      <origin xyz="0.222 0.155 0.109" rpy="${90*d2r} 0 ${240*d2r}"/>
     </xacro:thruster_macro>
     <xacro:thruster_macro namespace="${namespace}" thruster_id="6">
-      <origin xyz="-0.281372 -0.150723 0.145563" rpy="0 0 ${-25*d2r}"/>
+      <origin xyz="-0.222 -0.155 0.109" rpy="${90*d2r} 0 ${60*d2r}"/>
     </xacro:thruster_macro>
     <xacro:thruster_macro namespace="${namespace}" thruster_id="7">
-      <origin xyz="0.193622 -0.200534 0.145563" rpy="0 0 ${-25*d2r}"/>
-    </xacro:thruster_macro> -->
+      <origin xyz="0.222 -0.155 0.109" rpy="${90*d2r} 0 ${120*d2r}"/>
+    </xacro:thruster_macro>
     <!-- Instantiate fins, if necessary -->
     <!-- <xacro:fin_macro namespace="${namespace}" fin_id="0">

Commit message: Mid-change with thruster orientation. Might have fixed weird corner error bug that stopped the gzclient when reuploading the sub by fixing inertial dimensions of thruster. Still figuring out transparency of hull

File: simulation/mantaray_description/urdf/actuators.xacro (robot description, xacro)
@@ -12,8 +12,7 @@
       <origin xyz="-0.25 -0.34 0.244899" rpy="0 ${90*d2r} 0"/>
     </xacro:thruster_macro>
-    <xacro:thruster_macro namespace="${namespace}" thruster_id="1">
+    <!-- <xacro:thruster_macro namespace="${namespace}" thruster_id="1">
       <origin xyz="0.25 -0.34 0.244899" rpy="0 ${90*d2r} 0"/>
     </xacro:thruster_macro>
-                                    <!-- 0.238 -0.294170 0.244899 -->
     <xacro:thruster_macro namespace="${namespace}" thruster_id="2">
       <origin xyz="0.25 0.34 0.244899" rpy="0 ${90*d2r} 0"/>
@@ -33,5 +32,5 @@
     <xacro:thruster_macro namespace="${namespace}" thruster_id="7">
       <origin xyz="0.222 -0.155 0.109" rpy="${90*d2r} 0 ${120*d2r}"/>
-    </xacro:thruster_macro>
+    </xacro:thruster_macro> -->
     <!-- Instantiate fins, if necessary -->
     <!-- <xacro:fin_macro namespace="${namespace}" fin_id="0">

File: simulation/mantaray_description/urdf/base.xacro (robot description, xacro)
@@ -37,7 +37,8 @@
           <origin xyz="${cog}" rpy="0 0 0"/>
           <inertia ixx="1.313975" ixy="-0.008298" ixz=".021249" iyy="1.633282" iyz="0.0002475" izz="0.546458"/> <!-- From RexRov2 -->
-      </inertial>
+        </inertial>
       <!-- Units are in kg * meters^2 -->
         <visual name='visual'>
+          <transparency>0.8</transparency>
           <origin xyz="0 0 0.204636" rpy="0 0 0"/>
           <geometry>

File: simulation/mantaray_description/urdf/snippets.xacro (robot description, xacro)
@@ -21,5 +21,5 @@
     </joint>
     <link name="${namespace}/thruster_${thruster_id}">
-      <xacro:box_inertial x="0" y="0" z="0" mass="0.001">
+      <xacro:box_inertial x="113" y="97" z="97" mass="0.344"> <!--Mass in air is 344 g and in water is 156g-->
         <origin xyz="0 0 0" rpy="0 0 0"/>
       </xacro:box_inertial>

Commit message: Added changes to the transformation of the thrusters.

File: simulation/mantaray_description/urdf/actuators.xacro (robot description, xacro)
@@ -10,27 +10,27 @@
     <!-- Taken from RexRov2-->
     <xacro:thruster_macro namespace="${namespace}" thruster_id="0"> <!-- I inputed-->
-      <origin xyz="-0.25 -0.34 0.244899" rpy="0 ${90*d2r} 0"/>
+      <origin xyz="-0.23 -0.333 0.118" rpy="${90*d2r} 0 ${300*d2r}"/>
     </xacro:thruster_macro>
-    <!-- <xacro:thruster_macro namespace="${namespace}" thruster_id="1">
-      <origin xyz="0.25 -0.34 0.244899" rpy="0 ${90*d2r} 0"/>
+    <xacro:thruster_macro namespace="${namespace}" thruster_id="1">
+      <origin xyz="0.23 -0.333 0.118" rpy="${90*d2r} 0 ${240*d2r}"/>
     </xacro:thruster_macro>
     <xacro:thruster_macro namespace="${namespace}" thruster_id="2">
-      <origin xyz="0.25 0.34 0.244899" rpy="0 ${90*d2r} 0"/>
+      <origin xyz="0.23 0.333 0.118" rpy="${90*d2r} 0 ${20*d2r}"/>
     </xacro:thruster_macro>
     <xacro:thruster_macro namespace="${namespace}" thruster_id="3">
-      <origin xyz="-0.25 0.34 0.244899" rpy="0 ${90*d2r} 0"/>
+      <origin xyz="-0.23 0.3333 0.118" rpy="${90*d2r} 0 ${160*d2r}"/>
     </xacro:thruster_macro>
     <xacro:thruster_macro namespace="${namespace}" thruster_id="4">
-      <origin xyz="-0.222 0.155 0.109" rpy="${90*d2r} 0 ${300*d2r}"/>
+      <origin xyz="-0.222 0.155 0.109" rpy="0 ${90*d2r} 0"/>
     </xacro:thruster_macro>
     <xacro:thruster_macro namespace="${namespace}" thruster_id="5">
-      <origin xyz="0.222 0.155 0.109" rpy="${90*d2r} 0 ${240*d2r}"/>
+      <origin xyz="0.222 0.155 0.109" rpy="0 ${90*d2r} 0"/>
     </xacro:thruster_macro>
     <xacro:thruster_macro namespace="${namespace}" thruster_id="6">
-      <origin xyz="-0.222 -0.155 0.109" rpy="${90*d2r} 0 ${60*d2r}"/>
+      <origin xyz="-0.222 -0.155 0.109" rpy="0 ${90*d2r} 0"/>
     </xacro:thruster_macro>
     <xacro:thruster_macro namespace="${namespace}" thruster_id="7">
-      <origin xyz="0.222 -0.155 0.109" rpy="${90*d2r} 0 ${120*d2r}"/>
-    </xacro:thruster_macro> -->
+      <origin xyz="0.222 -0.155 0.109" rpy="0 ${90*d2r} 0"/>
+    </xacro:thruster_macro>
     <!-- Instantiate fins, if necessary -->
     <!-- <xacro:fin_macro namespace="${namespace}" fin_id="0">

File: simulation/mantaray_description/urdf/snippets.xacro (robot description, xacro)
@@ -27,5 +27,5 @@
         <origin rpy="0 0 0" xyz="0 0 0"/>
         <geometry>
-          <mesh filename="${prop_mesh_file}" scale="1 1 1"/>
+          <mesh filename="${prop_mesh_file}" scale="0.9 0.9 0.9"/>
         </geometry>
       </visual>

Commit message: William and Matt fixed the sim thruster issuegit add --all

File: simulation/mantaray_description/urdf/actuators.xacro (robot description, xacro)
@@ -22,14 +22,14 @@
     </xacro:thruster_macro>
     <xacro:thruster_macro namespace="${namespace}" thruster_id="4">
-      <origin xyz="-0.25 0.2 0.15" rpy="0 ${270*d2r} 0"/>
+      <origin xyz="-0.25 0.2 0.15" rpy="0 ${90*d2r} 0"/>
     </xacro:thruster_macro>
     <xacro:thruster_macro namespace="${namespace}" thruster_id="5">
-      <origin xyz="0.25 0.2 0.15" rpy="0 ${270*d2r} 0"/>
+      <origin xyz="0.25 0.2 0.15" rpy="0 ${90*d2r} 0"/>
     </xacro:thruster_macro>
     <xacro:thruster_macro namespace="${namespace}" thruster_id="6">
-      <origin xyz="-0.25 -0.2 0.15" rpy="0 ${270*d2r} 0"/>
+      <origin xyz="-0.25 -0.2 0.15" rpy="0 ${90*d2r} 0"/>
     </xacro:thruster_macro>
     <xacro:thruster_macro namespace="${namespace}" thruster_id="7">
-      <origin xyz="0.25 -0.2 0.15" rpy="0 ${270*d2r} 0"/>
+      <origin xyz="0.25 -0.2 0.15" rpy="0 ${90*d2r} 0"/>
     </xacro:thruster_macro>
     <!-- Instantiate fins, if necessary -->

File: simulation/mantaray_description/urdf/base.xacro (robot description, xacro)
@@ -14,6 +14,8 @@
   <xacro:property name="mass" value="22.102392"/>
   <!-- Center of gravity -->
+  <!-- <xacro:property name="cog" value="1.8 -1.17088 -1.62"/> -->
   <xacro:property name="cog" value="0.000018 -0.017088 -0.000362"/>
   <!-- Fluid density -->
+  <!-- <xacro:property name="rho" value="1028"/> -->
   <xacro:property name="rho" value="1028"/>
   <!--
@@ -41,6 +43,6 @@
           <mass value="${mass}" />
           <origin xyz="${cog}" rpy="0 0 0"/>
-          <inertia ixx="1343.163" ixy="0.003" ixz="0.132" iyy="1793.012" iyz="0.084" izz="649.198"/>
-          <!-- <inertia ixx="1.343163" ixy="0.000003" ixz="0.000132" iyy="1.793012" iyz="0.000084" izz="0.649198"/>  -->
+          <!-- <inertia ixx="1343.163" ixy="0.003" ixz="0.132" iyy="1793.012" iyz="0.084" izz="649.198"/> -->
+          <inertia ixx="1.343163" ixy="0.000003" ixz="0.000132" iyy="1.793012" iyz="0.000084" izz="0.649198"/>
         </inertial>
       <!-- Units are in kg * meters^2 -->

File: simulation/mantaray_description/urdf/gazebo.xacro (robot description, xacro)
@@ -2,5 +2,6 @@
 <robot xmlns:xacro="http://www.ros.org/wiki/xacro">
     <!-- Center of buoyancy -->
-    <xacro:property name="mantaray_cob" value="0 0 0"/> <!-- Random value -->
+    <xacro:property name="mantaray_cob" value="0 0 0"/> Random value
+    <!-- <xacro:property name="mantaray_cob" value="1.8 -1.17088 -1.62"/> -->
     <!-- Vehicle's actual volume (Gazebo cannot compute the volume out of the mesh) -->
     <xacro:property name="mantaray_volume" value="0.0910564446"/> <!-- Taken from RexRov2-->

File: simulation/mantaray_description/urdf/sensors.xacro (robot description, xacro)
@@ -21,4 +21,5 @@
     inertial_reference_frame="${inertial_reference_frame}">
     <origin xyz="0 0 0" rpy="0 0 0"/>
+    <!-- <origin xyz="1.8 -1.17088 -1.62" rpy="0 0 0"/> -->
   </xacro:default_imu_macro>
   <!-- This is a temporary sensor. Eventually we will use IMU only, especially in message_to_tf -->

File: simulation/mantaray_description/urdf/snippets.xacro (robot description, xacro)
@@ -13,5 +13,5 @@
     be initialized in the actuators.xacro file.
   -->
-  <xacro:macro name="thruster_macro" params="namespace thruster_id *origin">
+  <!-- <xacro:macro name="thruster_macro" params="namespace thruster_id *origin">
     <joint name="${namespace}/thruster_${thruster_id}_joint" type="continuous">
       <xacro:insert_block name="origin"/>
@@ -21,5 +21,5 @@
     </joint>
     <link name="${namespace}/thruster_${thruster_id}">
-      <xacro:box_inertial x="113" y="97" z="97" mass="0.344"> <!--Mass in air is 344 g and in water is 156g-->
+      <xacro:box_inertial x="113" y="97" z="97" mass="0.344">
         <origin xyz="0 0 0" rpy="0 0 0"/>
       </xacro:box_inertial>
@@ -55,6 +55,6 @@
       <selfCollide>false</selfCollide>
     </gazebo>
-  </xacro:macro>
-  <!-- <xacro:macro name="thruster_macro"
+  </xacro:macro> -->
+  <xacro:macro name="thruster_macro"
     params="namespace thruster_id *origin">
     <xacro:thruster_module_first_order_basic_fcn_macro
@@ -66,5 +66,5 @@
       <xacro:insert_block name="origin"/>
     </xacro:thruster_module_first_order_basic_fcn_macro>
-  </xacro:macro> -->
+  </xacro:macro>
   <!-- Ask david about dynaic time constant -->
   <!-- Look at the datasheet for rotor constant -->
