Commit message: Created a zed-M camera in the simulation. The settings aren't exactly the same yet and their is a bug with visualizing the point cloud in rviz since I can't figure out how to set the frame id of the point cloud within the URDF. I thought of creating my own plugin to go around this, but that'll take too long so I'm going to ignore this issue. if it is a real problem, I'll just use the default depth camera from UUV Simulator

File: simulation/mantaray_description/urdf/sensors.xacro (robot description, xacro)
@@ -7,4 +7,5 @@
     more examples or add you own custom sensor units.
   -->
+  <xacro:property name="M_PI"     value="3.1415926535897931" />
   <!-- Mount a GPS. -->
   <!-- <xacro:default_gps namespace="${namespace}" parent_link="${namespace}/base_link" /> -->
@@ -29,13 +30,15 @@
     inertial_reference_frame="${inertial_reference_frame}" />
   <!-- Mount a camera  -->
-  <xacro:default_camera namespace="${namespace}" parent_link="${namespace}/base_link" suffix="">
+  <!-- <xacro:default_camera namespace="${namespace}" parent_link="${namespace}/base_link" suffix="">
     <origin xyz="0 -0.333 0.2" rpy="0 0 0"/>
-  </xacro:default_camera>
+  </xacro:default_camera> -->
+  <xacro:include filename="depth_camera.xacro" ns="mantaray/base_link"/>
+  <!-- <xacro:include filename="tutorial_camera.xacro"/> -->
   <!-- Downward Facing Camera -->
-  <!-- <xacro:default_camera
+  <xacro:default_camera
     namespace="${namespace}"
     parent_link="${namespace}/base_link"
-    suffix="right">
-    <origin xyz="1.15 -0.63 0.4" rpy="0 0.6 0.4"/>
-  </xacro:default_camera> -->
+    suffix="bottom">
+    <origin xyz="0 0 0" rpy="0 ${M_PI/2} 0"/>
+  </xacro:default_camera>
 </robot>
