Commit message: Added some more accurate measurements for the sub

File: simulation/mantaray_description/urdf/base.xacro (robot description, xacro)
@@ -14,5 +14,5 @@
   <xacro:property name="mass" value="1862.87"/> <!-- From RexRov2 -->
   <!-- Center of gravity -->
-  <xacro:property name="cog" value="0 0 0"/>
+  <xacro:property name="cog" value="0.003631 -0.019556 0.015242"/> <!-- A little forward and down -->
   <!-- Fluid density -->
   <xacro:property name="rho" value="1028"/>
@@ -36,6 +36,7 @@
           <mass value="${mass}" />
           <origin xyz="${cog}" rpy="0 0 0"/>
-          <inertia ixx="525.39" ixy="1.44" ixz="33.41" iyy="794.20" iyz="2.6" izz="691.23"/> <!-- From RexRov2 -->
+          <inertia ixx="1.313975" ixy="-0.008298" ixz=".021249" iyy="1.633282" iyz="0.0002475" izz="0.546458"/> <!-- From RexRov2 -->
       </inertial>
+      <!-- Units are in kg * meters^2 -->
         <visual name='visual'>
           <origin xyz="0 0 0.204636" rpy="0 0 0"/>

File: simulation/mantaray_description/urdf/snippets.xacro (robot description, xacro)
@@ -24,4 +24,6 @@
     </xacro:thruster_module_first_order_basic_fcn_macro>
   </xacro:macro>
+  <!-- Ask david about dynaic time constant -->
+  <!-- Look at the datasheet for rotor constant -->
   <!--                                                                      -->
   <!-- MACRO FOR FIN/RUDDER UNITS  -->

Commit message: Refactored some of the code and directly connected world and base_link using a new frame. Didn't fix anything or show anything useful in Rviz

File: simulation/mantaray_description/urdf/base.xacro (robot description, xacro)
@@ -28,5 +28,4 @@
       <!-- Rigid body description of the base link -->
       <link name="${namespace}/base_link">
-        <parent link="world"/>
         <!--
           Be careful to setup the coefficients for the inertial tensor,

Commit message: Added a dummy link, but still have to finish the modifications to fully integrate it. Oscillations seem to be better, but still not useable. Made it neutrally buoyant since it's less complex

File: simulation/mantaray_description/urdf/base.xacro (robot description, xacro)
@@ -12,7 +12,7 @@
     Vehicle's parameters (remember to enter the model parameters below)
   -->
-  <xacro:property name="mass" value="1862.87"/> <!-- From RexRov2 -->
+  <xacro:property name="mass" value="22.102392"/>
   <!-- Center of gravity -->
-  <xacro:property name="cog" value="0.003631 -0.019556 0.015242"/> <!-- A little forward and down -->
+  <xacro:property name="cog" value="0.000018 -0.017088 -0.000362"/>
   <!-- Fluid density -->
   <xacro:property name="rho" value="1028"/>
@@ -26,6 +26,11 @@
   <!-- Vehicle macro -->
   <xacro:macro name="mantaray_base" params="namespace *gazebo use_simplified_mesh inertial_reference_frame">
+    <link name="${namespace}/base_link"/>
+      <joint name="${namespace}/base_link_to_chassis" type="fixed">
+        <parent link="${namespace}/base_link"/>
+        <child link="${namespace}/chassis"/>
+      </joint>
       <!-- Rigid body description of the base link -->
-      <link name="${namespace}/base_link">
+      <link name="${namespace}/chassis">
         <!--
           Be careful to setup the coefficients for the inertial tensor,
@@ -36,5 +41,6 @@
           <mass value="${mass}" />
           <origin xyz="${cog}" rpy="0 0 0"/>
-          <inertia ixx="1.313975" ixy="-0.008298" ixz=".021249" iyy="1.633282" iyz="0.0002475" izz="0.546458"/> <!-- From RexRov2 -->
+          <inertia ixx="1343.163" ixy="0.003" ixz="0.132" iyy="1793.012" iyz="0.084" izz="649.198"/>
+          <!-- <inertia ixx="1.343163" ixy="0.000003" ixz="0.000132" iyy="1.793012" iyz="0.000084" izz="0.649198"/>  -->
         </inertial>
       <!-- Units are in kg * meters^2 -->

File: simulation/mantaray_description/urdf/gazebo.xacro (robot description, xacro)
@@ -4,5 +4,5 @@
     <xacro:property name="mantaray_cob" value="0 0 0"/> <!-- Random value -->
     <!-- Vehicle's actual volume (Gazebo cannot compute the volume out of the mesh) -->
-    <xacro:property name="mantaray_volume" value="1.83826"/> <!-- Taken from RexRov2-->
+    <xacro:property name="mantaray_volume" value="0.0910564446"/> <!-- Taken from RexRov2-->
     <!-- Describing the dimensions of the vehicle's bounding box -->
     <xacro:property name="mantaray_length" value="0.629158"/> <!-- Might have mixed up length and width-->
@@ -13,5 +13,5 @@
       <link name="${namespace}/base_link">
         <!-- This flag will make the link neutrally buoyant -->
-        <neutrally_buoyant>0</neutrally_buoyant>
+        <neutrally_buoyant>1</neutrally_buoyant>
         <!-- Link's volume -->
         <volume>${mantaray_volume}</volume>
@@ -37,10 +37,10 @@
           <type>fossen</type>
           <added_mass> <!-- Taken from RexRov2-->
-            779.79 -6.8773 -103.32  8.5426 -165.54 -7.8033
-           -6.8773    1222   51.29  409.44 -5.8488  62.726
-           -103.32   51.29  3659.9  6.1112 -386.42  10.774
-            8.5426  409.44  6.1112   534.9 -10.027  21.019
-           -165.54 -5.8488 -386.42 -10.027  842.69 -1.1162
-           -7.8033  62.726  10.775  21.019 -1.1162  224.32
+            0 0 0 0 0 0
+            0 0 0 0 0 0
+            0 0 0 0 0 0
+            0 0 0 0 0 0
+            0 0 0 0 0 0
+            0 0 0 0 0 0
        </added_mass>
           <!--

Commit message: Spent a few hours trying to get the zedM camera imported via the code for zed-ros-wrapper. Since the repo was made for ros-foxy, I tried to reconfigure the code on my own but it's too time consuming so I'm going to simply create my own camera class. This should be something to revisit in the future though since using the Zed API will be helpful.

File: simulation/mantaray_description/urdf/base.xacro (robot description, xacro)
@@ -48,5 +48,5 @@
       <!-- Units are in kg * meters^2 -->
         <visual name='visual'>
-          <transparency>0.8</transparency>
+          <transparency>1</transparency>
           <origin xyz="0 0 0.204636" rpy="0 0 0"/>
           <geometry>

File: simulation/mantaray_description/urdf/sensors.xacro (robot description, xacro)
@@ -29,7 +29,7 @@
     inertial_reference_frame="${inertial_reference_frame}" />
   <!-- Mount a camera  -->
-  <!-- <xacro:default_camera namespace="${namespace}" parent_link="${namespace}/base_link" suffix="">
-    <origin xyz="1.15 0 0.4" rpy="0 0 0"/>
-  </xacro:default_camera> -->
+  <xacro:default_camera namespace="${namespace}" parent_link="${namespace}/base_link" suffix="">
+    <origin xyz="0 -0.333 0.2" rpy="0 0 0"/>
+  </xacro:default_camera>
   <!-- Downward Facing Camera -->
   <!-- <xacro:default_camera

Commit message: In the middle of creating a thruster class that can be used for both the sim and irl. Reorganized the data for the T200 thrusters to make it more accessible.

File: simulation/mantaray_description/urdf/base.xacro (robot description, xacro)
@@ -43,5 +43,4 @@
           <mass value="${mass}" />
           <origin xyz="${cog}" rpy="0 0 0"/>
-          <!-- <inertia ixx="1343.163" ixy="0.003" ixz="0.132" iyy="1793.012" iyz="0.084" izz="649.198"/> -->
           <inertia ixx="1.343163" ixy="0.000003" ixz="0.000132" iyy="1.793012" iyz="0.000084" izz="0.649198"/>
         </inertial>

File: simulation/mantaray_description/urdf/depth_camera.xacro (robot description, xacro)
@@ -12,6 +12,8 @@
   <xacro:arg name="cam_pitch"     default="0.0" />
   <xacro:arg name="cam_yaw"       default="${M_PI/2}" />
+  <xacro:arg name="frame_id" value="$(arg namespace)/base_link" />
   <xacro:arg name="gnss_frame"    default="" />
   <xacro:property name="parent" value="$(arg namespace)/base_link" />
+  <xacro:property name="frame_id" value="$(arg namespace)/base_link" />
   <xacro:property name="baseline" value="0.06" />
   <xacro:property name="height" value="0.0265" />

File: simulation/mantaray_description/urdf/sensors.xacro (robot description, xacro)
@@ -33,12 +33,18 @@
     <origin xyz="0 -0.333 0.2" rpy="0 0 0"/>
   </xacro:default_camera> -->
-  <xacro:include filename="depth_camera.xacro" ns="mantaray/base_link"/>
+  <!-- <xacro:include filename="depth_camera.xacro" ns="mantaray/base_link"/> -->
+  <xacro:duo3d_camera
+    namespace="${namespace}"
+    parent_link="${namespace}/base_link">
+    <origin xyz="0.0 0.4 0.2" rpy="0 0 ${M_PI/2}"/>
+  </xacro:duo3d_camera>
   <!-- <xacro:include filename="tutorial_camera.xacro"/> -->
   <!-- Downward Facing Camera -->
-  <xacro:default_camera
+  <xacro:regular_camera_plugin_macro
     namespace="${namespace}"
     parent_link="${namespace}/base_link"
-    suffix="bottom">
+    suffix="bottom"
+    scale="0.2">
     <origin xyz="0 0 0" rpy="0 ${M_PI/2} 0"/>
-  </xacro:default_camera>
+  </xacro:regular_camera_plugin_macro>
 </robot>
