Commit message: In the middle of creating a thruster class that can be used for both the sim and irl. Reorganized the data for the T200 thrusters to make it more accessible.

File: simulation/mantaray_description/urdf/snippets.xacro (robot description, xacro)
@@ -9,4 +9,5 @@
   <!-- I stole this dae file from https://github.com/francisc0garcia/robdos_sim/blob/master/models/robdos_model_thrust.dae -->
   <xacro:property name="prop_mesh_file" value="file://$(find mantaray_description)/meshes/mantaray_prop.dae"/>
+  <xacro:property name="voltage" value='12'/>
   <!--
     Thruster macro with integration of joint and link. The thrusters should
@@ -58,5 +59,42 @@
   <xacro:macro name="thruster_macro"
     params="namespace thruster_id *origin">
-    <xacro:thruster_module_first_order_basic_fcn_macro
+    <xacro:generic_thruster_macro
+      namespace="${namespace}"
+      thruster_id="${thruster_id}"
+      mesh_filename="${mesh_filename}">
+      <xacro:insert_block name="origin"/>
+      <xacro:rotor_dyn_first_order_macro time_constant="0.15"/> <!-- https://discuss.bluerobotics.com/t/question-regarding-t200/997/3-->
+      <xacro:if value="${voltage == '10'}">
+        <xacro:thruster_cf_linear_interp_macro
+          input_values="1100.0 1104.0 1108.0 1112.0 1116.0 1120.0 1124.0 1128.0 1132.0 1136.0 1140.0 1144.0 1148.0 1152.0 1156.0 1160.0 1164.0 1168.0 1172.0 1176.0 1180.0 1184.0 1188.0 1192.0 1196.0 1200.0 1204.0 1208.0 1212.0 1216.0 1220.0 1224.0 1228.0 1232.0 1236.0 1240.0 1244.0 1248.0 1252.0 1256.0 1260.0 1264.0 1268.0 1272.0 1276.0 1280.0 1284.0 1288.0 1292.0 1296.0 1300.0 1304.0 1308.0 1312.0 1316.0 1320.0 1324.0 1328.0 1332.0 1336.0 1340.0 1344.0 1348.0 1352.0 1356.0 1360.0 1364.0 1368.0 1372.0 1376.0 1380.0 1384.0 1388.0 1392.0 1396.0 1400.0 1404.0 1408.0 1412.0 1416.0 1420.0 1424.0 1428.0 1432.0 1436.0 1440.0 1444.0 1448.0 1452.0 1456.0 1460.0 1464.0 1468.0 1472.0 1476.0 1480.0 1484.0 1488.0 1492.0 1496.0 1500.0 1504.0 1508.0 1512.0 1516.0 1520.0 1524.0 1528.0 1532.0 1536.0 1540.0 1544.0 1548.0 1552.0 1556.0 1560.0 1564.0 1568.0 1572.0 1576.0 1580.0 1584.0 1588.0 1592.0 1596.0 1600.0 1604.0 1608.0 1612.0 1616.0 1620.0 1624.0 1628.0 1632.0 1636.0 1640.0 1644.0 1648.0 1652.0 1656.0 1660.0 1664.0 1668.0 1672.0 1676.0 1680.0 1684.0 1688.0 1692.0 1696.0 1700.0 1704.0 1708.0 1712.0 1716.0 1720.0 1724.0 1728.0 1732.0 1736.0 1740.0 1744.0 1748.0 1752.0 1756.0 1760.0 1764.0 1768.0 1772.0 1776.0 1780.0 1784.0 1788.0 1792.0 1796.0 1800.0 1804.0 1808.0 1812.0 1816.0 1820.0 1824.0 1828.0 1832.0 1836.0 1840.0 1844.0 1848.0 1852.0 1856.0 1860.0 1864.0 1868.0 1872.0 1876.0 1880.0 1884.0 1888.0 1892.0 1896.0 1900.0"
+          output_values="-2.309539266666666 -2.30424736 -2.29517552 -2.28156776 -2.2226008 -2.18177752 -2.16363384 -2.1318824 -2.1092028000000003 -2.05477176 -2.0411639999999998 -1.98673296 -1.95498152 -1.927766 -1.89147864 -1.8370476000000002 -1.80983208 -1.7916883999999997 -1.75540104 -1.7145777599999998 -1.68282632 -1.65107488 -1.6193234399999998 -1.59210792 -1.55582056 -1.53767688 -1.50138952 -1.4696380800000002 -1.44242256 -1.41067112 -1.360776 -1.32902456 -1.31995272 -1.28820128 -1.25644984 -1.22016248 -1.18841104 -1.1657314399999998 -1.13851592 -1.09769264 -1.07501304 -1.05686936 -1.0160460800000002 -0.98883056 -0.97068688 -0.9298636 -0.907184 -0.8799684799999999 -0.8527529599999999 -0.8255374400000001 -0.79832192 -0.78017824 -0.75296272 -0.72121128 -0.69853168 -0.6713161599999999 -0.6531724799999999 -0.6304928799999999 -0.6123491999999999 -0.58059776 -0.55338224 -0.53070264 -0.5125589599999999 -0.48534344 -0.46719976 -0.44452016 -0.42184056 -0.39916096 -0.38101728 -0.35380176 -0.33565808 -0.31297847999999995 -0.2948348 -0.27669112 -0.2494756 -0.23586784 -0.21318824 -0.19958048 -0.18143679999999998 -0.16329312 -0.15422128000000002 -0.1360776 -0.11793392 -0.09979024 -0.08618248 -0.07257472 -0.06350288000000001 -0.05443104 -0.045359199999999995 -0.031751440000000006 0.0 0.0 0.0 0.0 0.0 0.0 0.0 0.0 0.0 0.0 0.0 0.0 0.0 0.0 0.0 0.0 0.0 0.0 0.0 0.0 0.0 0.04082328 0.054431040000000014 0.06803880000000001 0.07711064000000001 0.09071839999999999 0.10886208 0.12700576 0.14514944 0.16329312 0.1814368 0.2041164 0.22226008 0.24493968 0.26308336 0.29029888 0.31297847999999995 0.33565808 0.3628736 0.38555320000000004 0.41276872 0.44452016 0.46719976 0.49441528 0.5216308 0.54884632 0.58059776 0.60781328 0.63956472 0.68492392 0.7030675999999999 0.7257471999999999 0.7620345599999999 0.79832192 0.8255374400000001 0.8527529599999999 0.88904032 0.9207917599999998 0.94800728 0.9752228000000001 0.97068688 1.04779752 1.07501304 1.1113004 1.1657314399999998 1.18387512 1.20655472 1.23830616 1.27459352 1.31088088 1.3562400799999998 1.41067112 1.4288148 1.4787099199999998 1.5240691199999998 1.54674872 1.57850016 1.62385936 1.6556108 1.69189816 1.72818552 1.77354472 1.80076024 1.84611944 1.87787088 1.9141582400000003 1.99126888 1.9958048 2.05930768 2.09105912 2.1228105600000005 2.16816976 2.2135289600000005 2.2724959200000003 2.30424736 2.3632143200000004 2.40857352 2.45393272 2.4811482400000004 2.5537229600000004 2.5809384800000004 2.61722584 2.6489772800000004 2.68526464 2.73515976 2.77144712 2.8213422400000003 2.87577328 2.8939169600000003 2.9165965600000003 2.9256683999999997"/>
+      </xacro:if>
+      <xacro:if value="${voltage == '12'}">
+        <xacro:thruster_cf_linear_interp_macro
+          input_values="1100.0 1104.0 1108.0 1112.0 1116.0 1120.0 1124.0 1128.0 1132.0 1136.0 1140.0 1144.0 1148.0 1152.0 1156.0 1160.0 1164.0 1168.0 1172.0 1176.0 1180.0 1184.0 1188.0 1192.0 1196.0 1200.0 1204.0 1208.0 1212.0 1216.0 1220.0 1224.0 1228.0 1232.0 1236.0 1240.0 1244.0 1248.0 1252.0 1256.0 1260.0 1264.0 1268.0 1272.0 1276.0 1280.0 1284.0 1288.0 1292.0 1296.0 1300.0 1304.0 1308.0 1312.0 1316.0 1320.0 1324.0 1328.0 1332.0 1336.0 1340.0 1344.0 1348.0 1352.0 1356.0 1360.0 1364.0 1368.0 1372.0 1376.0 1380.0 1384.0 1388.0 1392.0 1396.0 1400.0 1404.0 1408.0 1412.0 1416.0 1420.0 1424.0 1428.0 1432.0 1436.0 1440.0 1444.0 1448.0 1452.0 1456.0 1460.0 1464.0 1468.0 1472.0 1476.0 1480.0 1484.0 1488.0 1492.0 1496.0 1500.0 1504.0 1508.0 1512.0 1516.0 1520.0 1524.0 1528.0 1532.0 1536.0 1540.0 1544.0 1548.0 1552.0 1556.0 1560.0 1564.0 1568.0 1572.0 1576.0 1580.0 1584.0 1588.0 1592.0 1596.0 1600.0 1604.0 1608.0 1612.0 1616.0 1620.0 1624.0 1628.0 1632.0 1636.0 1640.0 1644.0 1648.0 1652.0 1656.0 1660.0 1664.0 1668.0 1672.0 1676.0 1680.0 1684.0 1688.0 1692.0 1696.0 1700.0 1704.0 1708.0 1712.0 1716.0 1720.0 1724.0 1728.0 1732.0 1736.0 1740.0 1744.0 1748.0 1752.0 1756.0 1760.0 1764.0 1768.0 1772.0 1776.0 1780.0 1784.0 1788.0 1792.0 1796.0 1800.0 1804.0 1808.0 1812.0 1816.0 1820.0 1824.0 1828.0 1832.0 1836.0 1840.0 1844.0 1848.0 1852.0 1856.0 1860.0 1864.0 1868.0 1872.0 1876.0 1880.0 1884.0 1888.0 1892.0 1896.0 1900.0"
+          output_values="-2.9037447866666666 -2.91659656 -2.89391696 -2.83041408 -2.78505488 -2.76237528 -2.721552 -2.67165688 -2.59908216 -2.59454624 -2.5627948000000003 -2.494756 -2.44032496 -2.43125312 -2.38589392 -2.34053472 -2.30424736 -2.25435224 -2.22713672 -2.18177752 -2.14095424 -2.09559504 -2.06837952 -2.00941256 -1.98219704 -1.94590968 -1.8824067999999998 -1.84611944 -1.80529616 -1.77808064 -1.73272144 -1.66468264 -1.65107488 -1.6102516000000002 -1.56035648 -1.53314096 -1.49231768 -1.4696380800000002 -1.43788664 -1.39706336 -1.36984784 -1.33356048 -1.2927372 -1.27912944 -1.22016248 -1.19294696 -1.15212368 -1.11583632 -1.08408488 -1.0432616 -1.0205819999999999 -0.99336648 -0.96161504 -0.9298636 -0.90264808 -0.87089664 -0.83460928 -0.793786 -0.7711064000000001 -0.7393549599999999 -0.72121128 -0.69399576 -0.6577084 -0.63956472 -0.60327736 -0.57152592 -0.5443104 -0.5170948799999999 -0.49441528 -0.47173568 -0.43998424 -0.41730464 -0.39008912 -0.36740952 -0.340194 -0.31751440000000003 -0.2948348 -0.26761928 -0.24493968 -0.226796 -0.2041164 -0.17690088 -0.16329312 -0.14514944 -0.12246984 -0.10886208 -0.09071839999999999 -0.07257472 -0.05896696 -0.045359199999999995 -0.03628736 0.0 0.0 0.0 0.0 0.0 0.0 0.0 0.0 0.0 0.0 0.0 0.0 0.0 0.0 0.0 0.0 0.0 0.0 0.0 0.04082328 0.05443104 0.07257472 0.09525432 0.113398 0.13154168000000002 0.15422128000000002 0.17690088 0.19958048 0.22226008 0.25401152000000005 0.27669112 0.30844256000000003 0.33112216 0.36740952 0.39462504 0.42637648 0.45812792 0.48987936 0.5170948799999999 0.54884632 0.5896696 0.62595696 0.6531724799999999 0.68492392 0.7121394400000001 0.75749864 0.78925008 0.83007336 0.8572888799999999 0.89357624 0.9298636 0.96615096 1.00243832 1.0387256799999998 1.0840848799999998 1.13851592 1.1611955199999997 1.19748288 1.23377024 1.27912944 1.3108808799999998 1.35170416 1.40159928 1.4333507199999995 1.4832458399999997 1.5286050399999995 1.5648924 1.6329311999999998 1.67375448 1.7100418399999997 1.7690088 1.81890392 1.84611944 1.9050863999999998 1.92323008 1.96405336 2.03209216 2.0865232 2.1318824 2.1772416 2.23620856 2.27249592 2.33146288 2.39950168 2.46300456 2.5083637599999995 2.5627948 2.61722584 2.6535132000000003 2.71248016 2.77598304 2.84402184 2.87123736 2.93020432 3.00731496 3.04360232 3.0844256000000003 3.15700032 3.22503912 3.26132648 3.31575752 3.3792603999999997 3.40194 3.4472992 3.50173024 3.56976904 3.63780784 3.70584664 3.69223888 3.7141624933333337"/>
+      </xacro:if>
+      <xacro:if value="${voltage == '14'}">
+        <xacro:thruster_cf_linear_interp_macro
+          input_values="1100.0 1104.0 1108.0 1112.0 1116.0 1120.0 1124.0 1128.0 1132.0 1136.0 1140.0 1144.0 1148.0 1152.0 1156.0 1160.0 1164.0 1168.0 1172.0 1176.0 1180.0 1184.0 1188.0 1192.0 1196.0 1200.0 1204.0 1208.0 1212.0 1216.0 1220.0 1224.0 1228.0 1232.0 1236.0 1240.0 1244.0 1248.0 1252.0 1256.0 1260.0 1264.0 1268.0 1272.0 1276.0 1280.0 1284.0 1288.0 1292.0 1296.0 1300.0 1304.0 1308.0 1312.0 1316.0 1320.0 1324.0 1328.0 1332.0 1336.0 1340.0 1344.0 1348.0 1352.0 1356.0 1360.0 1364.0 1368.0 1372.0 1376.0 1380.0 1384.0 1388.0 1392.0 1396.0 1400.0 1404.0 1408.0 1412.0 1416.0 1420.0 1424.0 1428.0 1432.0 1436.0 1440.0 1444.0 1448.0 1452.0 1456.0 1460.0 1464.0 1468.0 1472.0 1476.0 1480.0 1484.0 1488.0 1492.0 1496.0 1500.0 1504.0 1508.0 1512.0 1516.0 1520.0 1524.0 1528.0 1532.0 1536.0 1540.0 1544.0 1548.0 1552.0 1556.0 1560.0 1564.0 1568.0 1572.0 1576.0 1580.0 1584.0 1588.0 1592.0 1596.0 1600.0 1604.0 1608.0 1612.0 1616.0 1620.0 1624.0 1628.0 1632.0 1636.0 1640.0 1644.0 1648.0 1652.0 1656.0 1660.0 1664.0 1668.0 1672.0 1676.0 1680.0 1684.0 1688.0 1692.0 1696.0 1700.0 1704.0 1708.0 1712.0 1716.0 1720.0 1724.0 1728.0 1732.0 1736.0 1740.0 1744.0 1748.0 1752.0 1756.0 1760.0 1764.0 1768.0 1772.0 1776.0 1780.0 1784.0 1788.0 1792.0 1796.0 1800.0 1804.0 1808.0 1812.0 1816.0 1820.0 1824.0 1828.0 1832.0 1836.0 1840.0 1844.0 1848.0 1852.0 1856.0 1860.0 1864.0 1868.0 1872.0 1876.0 1880.0 1884.0 1888.0 1892.0 1896.0 1900.0"
+          output_values="-3.5168499733333336 -3.49719432 -3.4926584000000003 -3.45183512 -3.40194 -3.3565808 -3.29307792 -3.24771872 -3.18875176 -3.13885664 -3.09803336 -3.0572100799999995 -3.00277904 -2.93927616 -2.88484512 -2.84855776 -2.78051896 -2.76237528 -2.68980056 -2.64444136 -2.59454624 -2.52650744 -2.49022008 -2.45393272 -2.40857352 -2.34960656 -2.3359988 -2.25888816 -2.20445712 -2.1772416 -2.11827464 -2.0547717599999995 -2.02755624 -1.98673296 -1.90962232 -1.89147864 -1.81890392 -1.76447288 -1.71911368 -1.6828263200000002 -1.6329312 -1.57850016 -1.5648924 -1.5195332000000001 -1.47870992 -1.44242256 -1.40159928 -1.36984784 -1.3244886400000002 -1.28366536 -1.23830616 -1.1929469600000002 -1.16573144 -1.12490816 -1.0886208000000002 -1.0523334400000002 -1.0160460800000002 -0.98429464 -0.9525431999999999 -0.91625584 -0.8845044 -0.84821704 -0.80739376 -0.7665704799999999 -0.7393549599999999 -0.7030675999999999 -0.680388 -0.6486365599999999 -0.62142104 -0.58513368 -0.54884632 -0.5170948799999999 -0.48987936 -0.46266384 -0.42637648 -0.39916096 -0.37194544 -0.34926584 -0.31751440000000003 -0.28576296 -0.25854744 -0.23586784 -0.20865232 -0.18597272 -0.16329312 -0.14514943999999996 -0.12246984 -0.09979024 -0.08164655999999999 -0.0680388 -0.045359199999999995 -0.031751440000000006 0.0 0.0 0.0 0.0 0.0 0.0 0.0 0.0 0.0 0.0 0.0 0.0 0.0 0.0 0.0 0.0 0.0 0.0453592 0.06350288000000001 0.08164656 0.09979024 0.12246983999999997 0.14514944 0.17690087999999998 0.19958048 0.226796 0.26308336 0.29029888 0.32658624 0.3628736 0.39462504 0.42637648 0.46266384 0.4989512 0.53070264 0.57606184 0.62142104 0.64410064 0.68945984 0.7257471999999999 0.7665704799999999 0.8255374400000001 0.84821704 0.88904032 0.9207917599999998 0.96615096 0.9979024 1.05233344 1.09315672 1.14305184 1.2020188 1.23377024 1.27912944 1.32448864 1.36531192 1.4061351999999998 1.46056624 1.51046136 1.55128464 1.60571568 1.65107488 1.71004184 1.75993696 1.814368 1.85065536 1.9096223200000004 1.96405336 2.0048766400000004 2.0865232 2.1182746400000005 2.15909792 2.2452804 2.26796 2.34053472 2.4267172 2.50382784 2.5627948000000003 2.63536952 2.6580491200000003 2.75783936 2.78051896 2.8803092 2.9347402400000004 2.9937072 3.04813824 3.1297848 3.18875176 3.23411096 3.32482936 3.36111672 3.42008368 3.4926584000000003 3.5652331200000003 3.62420008 3.68770296 3.76934952 3.837388320000001 3.9235708 3.982537760000001 4.0278969600000005 4.10954352 4.15490272 4.21386968 4.30458808 4.38169872 4.422522 4.5087044800000005 4.52684816 4.5238242133333335"/>
+      </xacro:if>
+      <xacro:if value="${voltage == '16'}">
+        <xacro:thruster_cf_linear_interp_macro
+          input_values="1100.0 1104.0 1108.0 1112.0 1116.0 1120.0 1124.0 1128.0 1132.0 1136.0 1140.0 1144.0 1148.0 1152.0 1156.0 1160.0 1164.0 1168.0 1172.0 1176.0 1180.0 1184.0 1188.0 1192.0 1196.0 1200.0 1204.0 1208.0 1212.0 1216.0 1220.0 1224.0 1228.0 1232.0 1236.0 1240.0 1244.0 1248.0 1252.0 1256.0 1260.0 1264.0 1268.0 1272.0 1276.0 1280.0 1284.0 1288.0 1292.0 1296.0 1300.0 1304.0 1308.0 1312.0 1316.0 1320.0 1324.0 1328.0 1332.0 1336.0 1340.0 1344.0 1348.0 1352.0 1356.0 1360.0 1364.0 1368.0 1372.0 1376.0 1380.0 1384.0 1388.0 1392.0 1396.0 1400.0 1404.0 1408.0 1412.0 1416.0 1420.0 1424.0 1428.0 1432.0 1436.0 1440.0 1444.0 1448.0 1452.0 1456.0 1460.0 1464.0 1468.0 1472.0 1476.0 1480.0 1484.0 1488.0 1492.0 1496.0 1500.0 1504.0 1508.0 1512.0 1516.0 1520.0 1524.0 1528.0 1532.0 1536.0 1540.0 1544.0 1548.0 1552.0 1556.0 1560.0 1564.0 1568.0 1572.0 1576.0 1580.0 1584.0 1588.0 1592.0 1596.0 1600.0 1604.0 1608.0 1612.0 1616.0 1620.0 1624.0 1628.0 1632.0 1636.0 1640.0 1644.0 1648.0 1652.0 1656.0 1660.0 1664.0 1668.0 1672.0 1676.0 1680.0 1684.0 1688.0 1692.0 1696.0 1700.0 1704.0 1708.0 1712.0 1716.0 1720.0 1724.0 1728.0 1732.0 1736.0 1740.0 1744.0 1748.0 1752.0 1756.0 1760.0 1764.0 1768.0 1772.0 1776.0 1780.0 1784.0 1788.0 1792.0 1796.0 1800.0 1804.0 1808.0 1812.0 1816.0 1820.0 1824.0 1828.0 1832.0 1836.0 1840.0 1844.0 1848.0 1852.0 1856.0 1860.0 1864.0 1868.0 1872.0 1876.0 1880.0 1884.0 1888.0 1892.0 1896.0 1900.0"
+          output_values="-4.069476226666667 -4.05057656 -4.023361039999998 -3.96439408 -3.9008912000000002 -3.86913976 -3.82378056 -3.80110096 -3.75120584 -3.71491848 -3.65595152 -3.58791272 -3.51987392 -3.45183512 -3.3974040800000003 -3.3112216 -3.25225464 -3.20235952 -3.1071052000000003 -3.0390664000000003 -2.9937072 -2.9392761600000004 -2.86216552 -2.82134224 -2.77144712 -2.70794424 -2.6580491200000003 -2.5809384800000004 -2.54918704 -2.50836376 -2.45393272 -2.381358 -2.35414248 -2.27703184 -2.23620856 -2.19538528 -2.11827464 -2.08198728 -2.02302032 -1.97766112 -1.94137376 -1.8597272 -1.814368 -1.76447288 -1.70097 -1.66921856 -1.6102516000000002 -1.55582056 -1.51499728 -1.4877817599999998 -1.43788664 -1.39706336 -1.34716824 -1.30180904 -1.25644984 -1.2020188 -1.16119552 -1.12037224 -1.10222856 -1.05233344 -1.0205819999999999 -0.97975872 -0.94347136 -0.90264808 -0.87089664 -0.82100152 -0.7847141599999999 -0.7438908799999999 -0.71667536 -0.680388 -0.6486365599999999 -0.6168851200000001 -0.58059776 -0.53977448 -0.5125589599999999 -0.48080752 -0.44452016 -0.41730464 -0.38555320000000004 -0.35380176 -0.32205032 -0.2948348 -0.25854744 -0.23586784 -0.20865232 -0.18143679999999998 -0.14968536000000002 -0.12700576000000002 -0.10432616 -0.08618248 -0.0680388 -0.04989512 -0.03628736 0.0 0.0 0.0 0.0 0.0 0.0 0.0 0.0 0.0 0.0 0.0 0.0 0.0 0.0 0.0 0.04082328 0.054431040000000014 0.07711064000000001 0.09979024 0.12700576 0.15422128 0.1814368 0.21772416 0.2494756 0.29029888 0.32205032 0.35833768 0.39916096 0.43544832 0.47173568 0.5125589599999999 0.5579181599999999 0.60327736 0.63956472 0.680388 0.72121128 0.77564232 0.8164656 0.87089664 0.907184 0.94800728 0.99336648 1.0341897599999998 1.09769264 1.14305184 1.18387512 1.23830616 1.27912944 1.32902456 1.38799152 1.43788664 1.48324584 1.53767688 1.587572 1.65107488 1.69189816 1.75993696 1.8234398400000005 1.87787088 1.93230192 1.99126888 2.04569992 2.1228105600000005 2.1772416000000003 2.21806488 2.2770318400000003 2.381358 2.43125312 2.5174355999999998 2.5764025600000005 2.6535132000000003 2.73062384 2.75783936 2.8394859200000004 2.88938104 2.97556352 3.05267416 3.1071052000000003 3.17060808 3.21596728 3.3021497600000003 3.37472448 3.42008368 3.51080208 3.6060564 3.68316704 3.73759808 3.81924464 3.88728344 3.95532224 4.0596483999999995 4.14583088 4.254692960000002 4.30458808 4.38169872 4.5087044800000005 4.52684816 4.649318 4.70828496 4.7853956 4.83529072 4.93054504 5.0121915999999995 5.07569448 5.14373328 5.17548472 5.22084392 5.245035493333333"/>
+      </xacro:if>
+      <xacro:if value="${voltage == '18'}">
+        <xacro:thruster_cf_linear_interp_macro
+          input_values="1100.0 1104.0 1108.0 1112.0 1116.0 1120.0 1124.0 1128.0 1132.0 1136.0 1140.0 1144.0 1148.0 1152.0 1156.0 1160.0 1164.0 1168.0 1172.0 1176.0 1180.0 1184.0 1188.0 1192.0 1196.0 1200.0 1204.0 1208.0 1212.0 1216.0 1220.0 1224.0 1228.0 1232.0 1236.0 1240.0 1244.0 1248.0 1252.0 1256.0 1260.0 1264.0 1268.0 1272.0 1276.0 1280.0 1284.0 1288.0 1292.0 1296.0 1300.0 1304.0 1308.0 1312.0 1316.0 1320.0 1324.0 1328.0 1332.0 1336.0 1340.0 1344.0 1348.0 1352.0 1356.0 1360.0 1364.0 1368.0 1372.0 1376.0 1380.0 1384.0 1388.0 1392.0 1396.0 1400.0 1404.0 1408.0 1412.0 1416.0 1420.0 1424.0 1428.0 1432.0 1436.0 1440.0 1444.0 1448.0 1452.0 1456.0 1460.0 1464.0 1468.0 1472.0 1476.0 1480.0 1484.0 1488.0 1492.0 1496.0 1500.0 1504.0 1508.0 1512.0 1516.0 1520.0 1524.0 1528.0 1532.0 1536.0 1540.0 1544.0 1548.0 1552.0 1556.0 1560.0 1564.0 1568.0 1572.0 1576.0 1580.0 1584.0 1588.0 1592.0 1596.0 1600.0 1604.0 1608.0 1612.0 1616.0 1620.0 1624.0 1628.0 1632.0 1636.0 1640.0 1644.0 1648.0 1652.0 1656.0 1660.0 1664.0 1668.0 1672.0 1676.0 1680.0 1684.0 1688.0 1692.0 1696.0 1700.0 1704.0 1708.0 1712.0 1716.0 1720.0 1724.0 1728.0 1732.0 1736.0 1740.0 1744.0 1748.0 1752.0 1756.0 1760.0 1764.0 1768.0 1772.0 1776.0 1780.0 1784.0 1788.0 1792.0 1796.0 1800.0 1804.0 1808.0 1812.0 1816.0 1820.0 1824.0 1828.0 1832.0 1836.0 1840.0 1844.0 1848.0 1852.0 1856.0 1860.0 1864.0 1868.0 1872.0 1876.0 1880.0 1884.0 1888.0 1892.0 1896.0 1900.0"
+          output_values="-4.59035104 -4.54499184 -4.5313840800000005 -4.47695304 -4.41798608 -4.34994728 -4.34541136 -4.16851048 -4.18211824 -4.1050076 -4.0369687999999995 -3.9916096 -3.91449896 -3.86006792 -3.8101727999999997 -3.71491848 -3.68316704 -3.55616128 -3.54255352 -3.4246196 -3.3565808 -3.2658624 -3.19328768 -3.09349744 -3.02999456 -2.95741984 -2.8803092 -2.84402184 -2.77598304 -2.6988724 -2.65804912 -2.5854744 -2.52650744 -2.47661232 -2.42218128 -2.36321432 -2.31785512 -2.25435224 -2.20899304 -2.15909792 -2.1092028 -2.0411639999999998 -1.9958048 -1.94137376 -1.8824068 -1.814368 -1.75993696 -1.7191136799999998 -1.6601467199999995 -1.6102516000000002 -1.5648924 -1.5195332000000001 -1.46510216 -1.42427888 -1.37891968 -1.32902456 -1.2745935199999998 -1.2246984 -1.17480328 -1.13398 -1.0840848799999998 -1.0477975199999998 -1.01151016 -0.9706868799999998 -0.9343995199999998 -0.89357624 -0.8572888799999999 -0.81192968 -0.7711064000000001 -0.73935496 -0.69853168 -0.6713161599999999 -0.6350288000000001 -0.5987414400000001 -0.5579181599999999 -0.53070264 -0.49441528 -0.46266384 -0.4309124 -0.39916096 -0.36740952 -0.33565808 -0.30390664 -0.2721552 -0.24040376 -0.20865232 -0.18143679999999998 -0.15422128000000002 -0.12700576000000002 -0.10432616 -0.07711064000000001 -0.05896696 -0.0453592 0.0 0.0 0.0 0.0 0.0 0.0 0.0 0.0 0.0 0.0 0.0 0.0 0.0 0.0 0.0 0.0453592 0.06803880000000001 0.09071839999999999 0.12246984 0.14968536000000002 0.18143679999999998 0.21318824 0.2494756 0.28576296 0.31751440000000003 0.35833768 0.39008912 0.42637648 0.47173568 0.5080230400000001 0.54884632 0.58513368 0.62595696 0.66678024 0.69853168 0.75749864 0.80285784 0.8391451999999999 0.8799684799999999 0.9162558399999998 0.96615096 1.01604608 1.0750130399999998 1.13398 1.1793391999999998 1.2246984 1.27912944 1.31995272 1.3834556 1.42427888 1.4877817599999998 1.5376768799999998 1.5966438399999998 1.6782903999999998 1.74179328 1.78715248 1.84158352 1.91869416 1.9731252000000001 2.0366280800000003 2.08198728 2.17270568 2.21806488 2.28156776 2.36321432 2.43125312 2.50382784 2.5854744 2.64444136 2.7442316000000004 2.79412672 2.8667014399999995 2.9256683999999997 3.01185088 3.10256928 3.14792848 3.20689544 3.2658624 3.39286816 3.45637104 3.5380176 3.628736 3.72399032 3.79202912 3.9235708 4.01882512 4.14129496 4.20933376 4.31819584 4.4089142400000005 4.53592 4.66746168 4.6946772 4.86250624 4.91693728 5.01672752 5.121053679999998 5.20723616 5.29341864 5.38413704 5.49753504 5.59732528 5.66536408 5.76969024 5.82412128 5.8966959999999995 5.98287848 6.016141893333334"/>
+      </xacro:if>
+      <xacro:if value="${voltage == '20'}">
+        <xacro:thruster_cf_linear_interp_macro
+          input_values="1100.0 1104.0 1108.0 1112.0 1116.0 1120.0 1124.0 1128.0 1132.0 1136.0 1140.0 1144.0 1148.0 1152.0 1156.0 1160.0 1164.0 1168.0 1172.0 1176.0 1180.0 1184.0 1188.0 1192.0 1196.0 1200.0 1204.0 1208.0 1212.0 1216.0 1220.0 1224.0 1228.0 1232.0 1236.0 1240.0 1244.0 1248.0 1252.0 1256.0 1260.0 1264.0 1268.0 1272.0 1276.0 1280.0 1284.0 1288.0 1292.0 1296.0 1300.0 1304.0 1308.0 1312.0 1316.0 1320.0 1324.0 1328.0 1332.0 1336.0 1340.0 1344.0 1348.0 1352.0 1356.0 1360.0 1364.0 1368.0 1372.0 1376.0 1380.0 1384.0 1388.0 1392.0 1396.0 1400.0 1404.0 1408.0 1412.0 1416.0 1420.0 1424.0 1428.0 1432.0 1436.0 1440.0 1444.0 1448.0 1452.0 1456.0 1460.0 1464.0 1468.0 1472.0 1476.0 1480.0 1484.0 1488.0 1492.0 1496.0 1500.0 1504.0 1508.0 1512.0 1516.0 1520.0 1524.0 1528.0 1532.0 1536.0 1540.0 1544.0 1548.0 1552.0 1556.0 1560.0 1564.0 1568.0 1572.0 1576.0 1580.0 1584.0 1588.0 1592.0 1596.0 1600.0 1604.0 1608.0 1612.0 1616.0 1620.0 1624.0 1628.0 1632.0 1636.0 1640.0 1644.0 1648.0 1652.0 1656.0 1660.0 1664.0 1668.0 1672.0 1676.0 1680.0 1684.0 1688.0 1692.0 1696.0 1700.0 1704.0 1708.0 1712.0 1716.0 1720.0 1724.0 1728.0 1732.0 1736.0 1740.0 1744.0 1748.0 1752.0 1756.0 1760.0 1764.0 1768.0 1772.0 1776.0 1780.0 1784.0 1788.0 1792.0 1796.0 1800.0 1804.0 1808.0 1812.0 1816.0 1820.0 1824.0 1828.0 1832.0 1836.0 1840.0 1844.0 1848.0 1852.0 1856.0 1860.0 1864.0 1868.0 1872.0 1876.0 1880.0 1884.0 1888.0 1892.0 1896.0 1900.0"
+          output_values="-5.035627186666667 -4.9577605600000005 -4.9214732 -4.84436256 -4.79446744 -4.7445723200000005 -4.68 -4.57674328 -4.46334528 -4.40437832 -4.34994728 -4.22747744 -4.15943864 -4.11861536 -4.018825120000002 -3.95532224 -3.88728344 -3.8101727999999997 -3.7103825600000007 -3.66048744 -3.55616128 -3.47905064 -3.3565808 -3.2885419999999996 -3.16153624 -3.12524888 -3.00277904 -2.94381208 -2.87123736 -2.77598304 -2.73515976 -2.67165688 -2.6036180799999995 -2.54465112 -2.49929192 -2.43578904 -2.4040376 -2.3133192000000005 -2.26342408 -2.1999212000000004 -2.14095424 -2.1092028 -2.0411639999999998 -1.96858928 -1.91415824 -1.85519128 -1.79622432 -1.72818552 -1.6737544800000002 -1.6374671200000002 -1.58303608 -1.5195332000000001 -1.4741739999999999 -1.4106711200000002 -1.3743837600000002 -1.3244886400000002 -1.2700576 -1.2201624800000002 -1.17026736 -1.1067644800000005 -1.0659412 -1.0205819999999999 -0.98883056 -0.94347136 -0.907184 -0.8754325599999999 -0.83007336 -0.78017824 -0.75296272 -0.71667536 -0.68945984 -0.6577084 -0.6304928799999999 -0.5896696 -0.5579181599999999 -0.53070264 -0.50348712 -0.47173568 -0.44452016 -0.41276872 -0.38555320000000004 -0.35833767999999994 -0.32205032 -0.2948348 -0.26308336 -0.23586784 -0.2041164 -0.17236496 -0.14514943999999996 -0.12246984 -0.09071839999999999 -0.07257472 -0.05443104 -0.03628736 0.0 0.0 0.0 0.0 0.0 0.0 0.0 0.0 0.0 0.0 0.0 0.0 0.0 0.0 0.05896696 0.08618248 0.11339799999999997 0.14968536000000002 0.18143679999999998 0.21318824 0.2494756 0.28576296 0.32205032 0.3628736 0.39008912 0.42637648 0.46719976 0.4989511999999999 0.5352385599999999 0.57152592 0.6078132799999999 0.63956472 0.66224432 0.69853168 0.7393549599999999 0.78017824 0.8164656 0.8618248 0.88904032 0.93439952 0.9752228000000001 1.0205819999999999 1.06140528 1.1203722399999998 1.17026736 1.22016248 1.27912944 1.31088088 1.37891968 1.43788664 1.52860504 1.5830360799999998 1.64200304 1.73725736 1.8007602399999998 1.84611944 1.91869416 1.98219704 2.06837952 2.11827464 2.1999212000000004 2.24981632 2.32692696 2.43578904 2.52197152 2.6081540000000003 2.66258504 2.76237528 2.82587816 2.90752472 2.9937072 3.05721008 3.13432072 3.2205032000000005 3.27947016 3.3565807999999997 3.44276328 3.54708944 3.6423437600000006 3.72399032 3.84646016 3.96439408 4.10047168 4.209333760000002 4.32726768 4.422522 4.5540636800000005 4.6992131200000005 4.82168296 4.93054504 5.02126344 5.143733280000001 5.20270024 5.39320888 5.520214640000002 5.62000488 5.710723280000002 5.81504944 5.92844744 6.059989120000001 6.128027920000001 6.25503368 6.36389576 6.45915008 6.554404400000001 6.6224432 6.72223344"/>
+      </xacro:if>
+    </xacro:generic_thruster_macro>
+    <!-- <xacro:thruster_module_first_order_basic_fcn_macro
       namespace="${namespace}"
       thruster_id="${thruster_id}"
@@ -65,5 +103,5 @@
       rotor_constant="0.026546960744430276">
       <xacro:insert_block name="origin"/>
-    </xacro:thruster_module_first_order_basic_fcn_macro>
+    </xacro:thruster_module_first_order_basic_fcn_macro> -->
   </xacro:macro>
   <!-- Ask david about dynaic time constant -->
