Commit message: Added a DVL., but I think it's currently bugged since you can only get the distance the sub is from the seabed and not the velocity. Unless you have to calculate this by hand, this is a bug that I'll look into and try to fix.

File: simulation/mantaray_description/urdf/bottom_camera.xacro (robot description, xacro)
@@ -4,5 +4,5 @@
     <parent link="mantaray/base_link"/>
     <child link="camera_link"/>
-    <origin xyz="0 0 0" rpy="0 ${pi/2} 0"/>
+    <origin xyz="0 0 0.1" rpy="0 ${pi/2} 0"/>
   </joint>
   <link name="camera_link">
@@ -40,4 +40,5 @@
           <plugin name="camera_controller" filename="libgazebo_ros_camera.so">
               <frame_name>camera_link_optical</frame_name>
+              <imageTopicName>bottom_camera</imageTopicName>
           </plugin>
       </sensor>

File: simulation/mantaray_description/urdf/sensors.xacro (robot description, xacro)
@@ -47,3 +47,17 @@
     <origin xyz="0 0 0" rpy="0 ${M_PI/2} 0"/>
   </xacro:wideangle_camera> -->
+  <!-- DVL -->
+  <xacro:dvl_plugin_macro
+    namespace="${namespace}"
+    suffix=""
+    parent_link="${namespace}/base_link"
+    topic="a50_dvl"
+    scale="0.9"
+    update_rate = "10"
+    reference_frame="${namespace}/base_link"
+    noise_sigma="0.001"
+    noise_amplitude="0"
+  >
+    <origin xyz="0 0.2 0.1" rpy="0 ${pi/2} 0"/>
+  </xacro:dvl_plugin_macro>
 </robot>

File: simulation/mantaray_description/urdf/snippets.xacro (robot description, xacro)
@@ -71,7 +71,7 @@
       </xacro:if> -->
       <!-- <xacro:if value="${voltage == '12'}"> -->
-      <xacro:thruster_cf_linear_interp_macro
+      <!-- <xacro:thruster_cf_linear_interp_macro
         input_values="1100.0 1104.0 1108.0 1112.0 1116.0 1120.0 1124.0 1128.0 1132.0 1136.0 1140.0 1144.0 1148.0 1152.0 1156.0 1160.0 1164.0 1168.0 1172.0 1176.0 1180.0 1184.0 1188.0 1192.0 1196.0 1200.0 1204.0 1208.0 1212.0 1216.0 1220.0 1224.0 1228.0 1232.0 1236.0 1240.0 1244.0 1248.0 1252.0 1256.0 1260.0 1264.0 1268.0 1272.0 1276.0 1280.0 1284.0 1288.0 1292.0 1296.0 1300.0 1304.0 1308.0 1312.0 1316.0 1320.0 1324.0 1328.0 1332.0 1336.0 1340.0 1344.0 1348.0 1352.0 1356.0 1360.0 1364.0 1368.0 1372.0 1376.0 1380.0 1384.0 1388.0 1392.0 1396.0 1400.0 1404.0 1408.0 1412.0 1416.0 1420.0 1424.0 1428.0 1432.0 1436.0 1440.0 1444.0 1448.0 1452.0 1456.0 1460.0 1464.0 1468.0 1472.0 1476.0 1480.0 1484.0 1488.0 1492.0 1496.0 1500.0 1504.0 1508.0 1512.0 1516.0 1520.0 1524.0 1528.0 1532.0 1536.0 1540.0 1544.0 1548.0 1552.0 1556.0 1560.0 1564.0 1568.0 1572.0 1576.0 1580.0 1584.0 1588.0 1592.0 1596.0 1600.0 1604.0 1608.0 1612.0 1616.0 1620.0 1624.0 1628.0 1632.0 1636.0 1640.0 1644.0 1648.0 1652.0 1656.0 1660.0 1664.0 1668.0 1672.0 1676.0 1680.0 1684.0 1688.0 1692.0 1696.0 1700.0 1704.0 1708.0 1712.0 1716.0 1720.0 1724.0 1728.0 1732.0 1736.0 1740.0 1744.0 1748.0 1752.0 1756.0 1760.0 1764.0 1768.0 1772.0 1776.0 1780.0 1784.0 1788.0 1792.0 1796.0 1800.0 1804.0 1808.0 1812.0 1816.0 1820.0 1824.0 1828.0 1832.0 1836.0 1840.0 1844.0 1848.0 1852.0 1856.0 1860.0 1864.0 1868.0 1872.0 1876.0 1880.0 1884.0 1888.0 1892.0 1896.0 1900.0"
-        output_values="-2.9037447866666666 -2.91659656 -2.89391696 -2.83041408 -2.78505488 -2.76237528 -2.721552 -2.67165688 -2.59908216 -2.59454624 -2.5627948000000003 -2.494756 -2.44032496 -2.43125312 -2.38589392 -2.34053472 -2.30424736 -2.25435224 -2.22713672 -2.18177752 -2.14095424 -2.09559504 -2.06837952 -2.00941256 -1.98219704 -1.94590968 -1.8824067999999998 -1.84611944 -1.80529616 -1.77808064 -1.73272144 -1.66468264 -1.65107488 -1.6102516000000002 -1.56035648 -1.53314096 -1.49231768 -1.4696380800000002 -1.43788664 -1.39706336 -1.36984784 -1.33356048 -1.2927372 -1.27912944 -1.22016248 -1.19294696 -1.15212368 -1.11583632 -1.08408488 -1.0432616 -1.0205819999999999 -0.99336648 -0.96161504 -0.9298636 -0.90264808 -0.87089664 -0.83460928 -0.793786 -0.7711064000000001 -0.7393549599999999 -0.72121128 -0.69399576 -0.6577084 -0.63956472 -0.60327736 -0.57152592 -0.5443104 -0.5170948799999999 -0.49441528 -0.47173568 -0.43998424 -0.41730464 -0.39008912 -0.36740952 -0.340194 -0.31751440000000003 -0.2948348 -0.26761928 -0.24493968 -0.226796 -0.2041164 -0.17690088 -0.16329312 -0.14514944 -0.12246984 -0.10886208 -0.09071839999999999 -0.07257472 -0.05896696 -0.045359199999999995 -0.03628736 0.0 0.0 0.0 0.0 0.0 0.0 0.0 0.0 0.0 0.0 0.0 0.0 0.0 0.0 0.0 0.0 0.0 0.0 0.0 0.04082328 0.05443104 0.07257472 0.09525432 0.113398 0.13154168000000002 0.15422128000000002 0.17690088 0.19958048 0.22226008 0.25401152000000005 0.27669112 0.30844256000000003 0.33112216 0.36740952 0.39462504 0.42637648 0.45812792 0.48987936 0.5170948799999999 0.54884632 0.5896696 0.62595696 0.6531724799999999 0.68492392 0.7121394400000001 0.75749864 0.78925008 0.83007336 0.8572888799999999 0.89357624 0.9298636 0.96615096 1.00243832 1.0387256799999998 1.0840848799999998 1.13851592 1.1611955199999997 1.19748288 1.23377024 1.27912944 1.3108808799999998 1.35170416 1.40159928 1.4333507199999995 1.4832458399999997 1.5286050399999995 1.5648924 1.6329311999999998 1.67375448 1.7100418399999997 1.7690088 1.81890392 1.84611944 1.9050863999999998 1.92323008 1.96405336 2.03209216 2.0865232 2.1318824 2.1772416 2.23620856 2.27249592 2.33146288 2.39950168 2.46300456 2.5083637599999995 2.5627948 2.61722584 2.6535132000000003 2.71248016 2.77598304 2.84402184 2.87123736 2.93020432 3.00731496 3.04360232 3.0844256000000003 3.15700032 3.22503912 3.26132648 3.31575752 3.3792603999999997 3.40194 3.4472992 3.50173024 3.56976904 3.63780784 3.70584664 3.69223888 3.7141624933333337"/>
+        output_values="-2.9037447866666666 -2.91659656 -2.89391696 -2.83041408 -2.78505488 -2.76237528 -2.721552 -2.67165688 -2.59908216 -2.59454624 -2.5627948000000003 -2.494756 -2.44032496 -2.43125312 -2.38589392 -2.34053472 -2.30424736 -2.25435224 -2.22713672 -2.18177752 -2.14095424 -2.09559504 -2.06837952 -2.00941256 -1.98219704 -1.94590968 -1.8824067999999998 -1.84611944 -1.80529616 -1.77808064 -1.73272144 -1.66468264 -1.65107488 -1.6102516000000002 -1.56035648 -1.53314096 -1.49231768 -1.4696380800000002 -1.43788664 -1.39706336 -1.36984784 -1.33356048 -1.2927372 -1.27912944 -1.22016248 -1.19294696 -1.15212368 -1.11583632 -1.08408488 -1.0432616 -1.0205819999999999 -0.99336648 -0.96161504 -0.9298636 -0.90264808 -0.87089664 -0.83460928 -0.793786 -0.7711064000000001 -0.7393549599999999 -0.72121128 -0.69399576 -0.6577084 -0.63956472 -0.60327736 -0.57152592 -0.5443104 -0.5170948799999999 -0.49441528 -0.47173568 -0.43998424 -0.41730464 -0.39008912 -0.36740952 -0.340194 -0.31751440000000003 -0.2948348 -0.26761928 -0.24493968 -0.226796 -0.2041164 -0.17690088 -0.16329312 -0.14514944 -0.12246984 -0.10886208 -0.09071839999999999 -0.07257472 -0.05896696 -0.045359199999999995 -0.03628736 0.0 0.0 0.0 0.0 0.0 0.0 0.0 0.0 0.0 0.0 0.0 0.0 0.0 0.0 0.0 0.0 0.0 0.0 0.0 0.04082328 0.05443104 0.07257472 0.09525432 0.113398 0.13154168000000002 0.15422128000000002 0.17690088 0.19958048 0.22226008 0.25401152000000005 0.27669112 0.30844256000000003 0.33112216 0.36740952 0.39462504 0.42637648 0.45812792 0.48987936 0.5170948799999999 0.54884632 0.5896696 0.62595696 0.6531724799999999 0.68492392 0.7121394400000001 0.75749864 0.78925008 0.83007336 0.8572888799999999 0.89357624 0.9298636 0.96615096 1.00243832 1.0387256799999998 1.0840848799999998 1.13851592 1.1611955199999997 1.19748288 1.23377024 1.27912944 1.3108808799999998 1.35170416 1.40159928 1.4333507199999995 1.4832458399999997 1.5286050399999995 1.5648924 1.6329311999999998 1.67375448 1.7100418399999997 1.7690088 1.81890392 1.84611944 1.9050863999999998 1.92323008 1.96405336 2.03209216 2.0865232 2.1318824 2.1772416 2.23620856 2.27249592 2.33146288 2.39950168 2.46300456 2.5083637599999995 2.5627948 2.61722584 2.6535132000000003 2.71248016 2.77598304 2.84402184 2.87123736 2.93020432 3.00731496 3.04360232 3.0844256000000003 3.15700032 3.22503912 3.26132648 3.31575752 3.3792603999999997 3.40194 3.4472992 3.50173024 3.56976904 3.63780784 3.70584664 3.69223888 3.7141624933333337"/> -->
       <!-- </xacro:if> -->
       <!-- <xacro:if value="${voltage == '14'}">
@@ -89,10 +89,10 @@
           input_values="1100.0 1104.0 1108.0 1112.0 1116.0 1120.0 1124.0 1128.0 1132.0 1136.0 1140.0 1144.0 1148.0 1152.0 1156.0 1160.0 1164.0 1168.0 1172.0 1176.0 1180.0 1184.0 1188.0 1192.0 1196.0 1200.0 1204.0 1208.0 1212.0 1216.0 1220.0 1224.0 1228.0 1232.0 1236.0 1240.0 1244.0 1248.0 1252.0 1256.0 1260.0 1264.0 1268.0 1272.0 1276.0 1280.0 1284.0 1288.0 1292.0 1296.0 1300.0 1304.0 1308.0 1312.0 1316.0 1320.0 1324.0 1328.0 1332.0 1336.0 1340.0 1344.0 1348.0 1352.0 1356.0 1360.0 1364.0 1368.0 1372.0 1376.0 1380.0 1384.0 1388.0 1392.0 1396.0 1400.0 1404.0 1408.0 1412.0 1416.0 1420.0 1424.0 1428.0 1432.0 1436.0 1440.0 1444.0 1448.0 1452.0 1456.0 1460.0 1464.0 1468.0 1472.0 1476.0 1480.0 1484.0 1488.0 1492.0 1496.0 1500.0 1504.0 1508.0 1512.0 1516.0 1520.0 1524.0 1528.0 1532.0 1536.0 1540.0 1544.0 1548.0 1552.0 1556.0 1560.0 1564.0 1568.0 1572.0 1576.0 1580.0 1584.0 1588.0 1592.0 1596.0 1600.0 1604.0 1608.0 1612.0 1616.0 1620.0 1624.0 1628.0 1632.0 1636.0 1640.0 1644.0 1648.0 1652.0 1656.0 1660.0 1664.0 1668.0 1672.0 1676.0 1680.0 1684.0 1688.0 1692.0 1696.0 1700.0 1704.0 1708.0 1712.0 1716.0 1720.0 1724.0 1728.0 1732.0 1736.0 1740.0 1744.0 1748.0 1752.0 1756.0 1760.0 1764.0 1768.0 1772.0 1776.0 1780.0 1784.0 1788.0 1792.0 1796.0 1800.0 1804.0 1808.0 1812.0 1816.0 1820.0 1824.0 1828.0 1832.0 1836.0 1840.0 1844.0 1848.0 1852.0 1856.0 1860.0 1864.0 1868.0 1872.0 1876.0 1880.0 1884.0 1888.0 1892.0 1896.0 1900.0"
           output_values="-4.59035104 -4.54499184 -4.5313840800000005 -4.47695304 -4.41798608 -4.34994728 -4.34541136 -4.16851048 -4.18211824 -4.1050076 -4.0369687999999995 -3.9916096 -3.91449896 -3.86006792 -3.8101727999999997 -3.71491848 -3.68316704 -3.55616128 -3.54255352 -3.4246196 -3.3565808 -3.2658624 -3.19328768 -3.09349744 -3.02999456 -2.95741984 -2.8803092 -2.84402184 -2.77598304 -2.6988724 -2.65804912 -2.5854744 -2.52650744 -2.47661232 -2.42218128 -2.36321432 -2.31785512 -2.25435224 -2.20899304 -2.15909792 -2.1092028 -2.0411639999999998 -1.9958048 -1.94137376 -1.8824068 -1.814368 -1.75993696 -1.7191136799999998 -1.6601467199999995 -1.6102516000000002 -1.5648924 -1.5195332000000001 -1.46510216 -1.42427888 -1.37891968 -1.32902456 -1.2745935199999998 -1.2246984 -1.17480328 -1.13398 -1.0840848799999998 -1.0477975199999998 -1.01151016 -0.9706868799999998 -0.9343995199999998 -0.89357624 -0.8572888799999999 -0.81192968 -0.7711064000000001 -0.73935496 -0.69853168 -0.6713161599999999 -0.6350288000000001 -0.5987414400000001 -0.5579181599999999 -0.53070264 -0.49441528 -0.46266384 -0.4309124 -0.39916096 -0.36740952 -0.33565808 -0.30390664 -0.2721552 -0.24040376 -0.20865232 -0.18143679999999998 -0.15422128000000002 -0.12700576000000002 -0.10432616 -0.07711064000000001 -0.05896696 -0.0453592 0.0 0.0 0.0 0.0 0.0 0.0 0.0 0.0 0.0 0.0 0.0 0.0 0.0 0.0 0.0 0.0453592 0.06803880000000001 0.09071839999999999 0.12246984 0.14968536000000002 0.18143679999999998 0.21318824 0.2494756 0.28576296 0.31751440000000003 0.35833768 0.39008912 0.42637648 0.47173568 0.5080230400000001 0.54884632 0.58513368 0.62595696 0.66678024 0.69853168 0.75749864 0.80285784 0.8391451999999999 0.8799684799999999 0.9162558399999998 0.96615096 1.01604608 1.0750130399999998 1.13398 1.1793391999999998 1.2246984 1.27912944 1.31995272 1.3834556 1.42427888 1.4877817599999998 1.5376768799999998 1.5966438399999998 1.6782903999999998 1.74179328 1.78715248 1.84158352 1.91869416 1.9731252000000001 2.0366280800000003 2.08198728 2.17270568 2.21806488 2.28156776 2.36321432 2.43125312 2.50382784 2.5854744 2.64444136 2.7442316000000004 2.79412672 2.8667014399999995 2.9256683999999997 3.01185088 3.10256928 3.14792848 3.20689544 3.2658624 3.39286816 3.45637104 3.5380176 3.628736 3.72399032 3.79202912 3.9235708 4.01882512 4.14129496 4.20933376 4.31819584 4.4089142400000005 4.53592 4.66746168 4.6946772 4.86250624 4.91693728 5.01672752 5.121053679999998 5.20723616 5.29341864 5.38413704 5.49753504 5.59732528 5.66536408 5.76969024 5.82412128 5.8966959999999995 5.98287848 6.016141893333334"/>
-      </xacro:if>
-      <xacro:if value="${voltage == '20'}">
-        <xacro:thruster_cf_linear_interp_macro
-          input_values="1100.0 1104.0 1108.0 1112.0 1116.0 1120.0 1124.0 1128.0 1132.0 1136.0 1140.0 1144.0 1148.0 1152.0 1156.0 1160.0 1164.0 1168.0 1172.0 1176.0 1180.0 1184.0 1188.0 1192.0 1196.0 1200.0 1204.0 1208.0 1212.0 1216.0 1220.0 1224.0 1228.0 1232.0 1236.0 1240.0 1244.0 1248.0 1252.0 1256.0 1260.0 1264.0 1268.0 1272.0 1276.0 1280.0 1284.0 1288.0 1292.0 1296.0 1300.0 1304.0 1308.0 1312.0 1316.0 1320.0 1324.0 1328.0 1332.0 1336.0 1340.0 1344.0 1348.0 1352.0 1356.0 1360.0 1364.0 1368.0 1372.0 1376.0 1380.0 1384.0 1388.0 1392.0 1396.0 1400.0 1404.0 1408.0 1412.0 1416.0 1420.0 1424.0 1428.0 1432.0 1436.0 1440.0 1444.0 1448.0 1452.0 1456.0 1460.0 1464.0 1468.0 1472.0 1476.0 1480.0 1484.0 1488.0 1492.0 1496.0 1500.0 1504.0 1508.0 1512.0 1516.0 1520.0 1524.0 1528.0 1532.0 1536.0 1540.0 1544.0 1548.0 1552.0 1556.0 1560.0 1564.0 1568.0 1572.0 1576.0 1580.0 1584.0 1588.0 1592.0 1596.0 1600.0 1604.0 1608.0 1612.0 1616.0 1620.0 1624.0 1628.0 1632.0 1636.0 1640.0 1644.0 1648.0 1652.0 1656.0 1660.0 1664.0 1668.0 1672.0 1676.0 1680.0 1684.0 1688.0 1692.0 1696.0 1700.0 1704.0 1708.0 1712.0 1716.0 1720.0 1724.0 1728.0 1732.0 1736.0 1740.0 1744.0 1748.0 1752.0 1756.0 1760.0 1764.0 1768.0 1772.0 1776.0 1780.0 1784.0 1788.0 1792.0 1796.0 1800.0 1804.0 1808.0 1812.0 1816.0 1820.0 1824.0 1828.0 1832.0 1836.0 1840.0 1844.0 1848.0 1852.0 1856.0 1860.0 1864.0 1868.0 1872.0 1876.0 1880.0 1884.0 1888.0 1892.0 1896.0 1900.0"
-          output_values="-5.035627186666667 -4.9577605600000005 -4.9214732 -4.84436256 -4.79446744 -4.7445723200000005 -4.68 -4.57674328 -4.46334528 -4.40437832 -4.34994728 -4.22747744 -4.15943864 -4.11861536 -4.018825120000002 -3.95532224 -3.88728344 -3.8101727999999997 -3.7103825600000007 -3.66048744 -3.55616128 -3.47905064 -3.3565808 -3.2885419999999996 -3.16153624 -3.12524888 -3.00277904 -2.94381208 -2.87123736 -2.77598304 -2.73515976 -2.67165688 -2.6036180799999995 -2.54465112 -2.49929192 -2.43578904 -2.4040376 -2.3133192000000005 -2.26342408 -2.1999212000000004 -2.14095424 -2.1092028 -2.0411639999999998 -1.96858928 -1.91415824 -1.85519128 -1.79622432 -1.72818552 -1.6737544800000002 -1.6374671200000002 -1.58303608 -1.5195332000000001 -1.4741739999999999 -1.4106711200000002 -1.3743837600000002 -1.3244886400000002 -1.2700576 -1.2201624800000002 -1.17026736 -1.1067644800000005 -1.0659412 -1.0205819999999999 -0.98883056 -0.94347136 -0.907184 -0.8754325599999999 -0.83007336 -0.78017824 -0.75296272 -0.71667536 -0.68945984 -0.6577084 -0.6304928799999999 -0.5896696 -0.5579181599999999 -0.53070264 -0.50348712 -0.47173568 -0.44452016 -0.41276872 -0.38555320000000004 -0.35833767999999994 -0.32205032 -0.2948348 -0.26308336 -0.23586784 -0.2041164 -0.17236496 -0.14514943999999996 -0.12246984 -0.09071839999999999 -0.07257472 -0.05443104 -0.03628736 0.0 0.0 0.0 0.0 0.0 0.0 0.0 0.0 0.0 0.0 0.0 0.0 0.0 0.0 0.05896696 0.08618248 0.11339799999999997 0.14968536000000002 0.18143679999999998 0.21318824 0.2494756 0.28576296 0.32205032 0.3628736 0.39008912 0.42637648 0.46719976 0.4989511999999999 0.5352385599999999 0.57152592 0.6078132799999999 0.63956472 0.66224432 0.69853168 0.7393549599999999 0.78017824 0.8164656 0.8618248 0.88904032 0.93439952 0.9752228000000001 1.0205819999999999 1.06140528 1.1203722399999998 1.17026736 1.22016248 1.27912944 1.31088088 1.37891968 1.43788664 1.52860504 1.5830360799999998 1.64200304 1.73725736 1.8007602399999998 1.84611944 1.91869416 1.98219704 2.06837952 2.11827464 2.1999212000000004 2.24981632 2.32692696 2.43578904 2.52197152 2.6081540000000003 2.66258504 2.76237528 2.82587816 2.90752472 2.9937072 3.05721008 3.13432072 3.2205032000000005 3.27947016 3.3565807999999997 3.44276328 3.54708944 3.6423437600000006 3.72399032 3.84646016 3.96439408 4.10047168 4.209333760000002 4.32726768 4.422522 4.5540636800000005 4.6992131200000005 4.82168296 4.93054504 5.02126344 5.143733280000001 5.20270024 5.39320888 5.520214640000002 5.62000488 5.710723280000002 5.81504944 5.92844744 6.059989120000001 6.128027920000001 6.25503368 6.36389576 6.45915008 6.554404400000001 6.6224432 6.72223344"/>
       </xacro:if> -->
+      <!-- <xacro:if value="${voltage == '20'}"> -->
+      <xacro:thruster_cf_linear_interp_macro
+        input_values="1100.0 1104.0 1108.0 1112.0 1116.0 1120.0 1124.0 1128.0 1132.0 1136.0 1140.0 1144.0 1148.0 1152.0 1156.0 1160.0 1164.0 1168.0 1172.0 1176.0 1180.0 1184.0 1188.0 1192.0 1196.0 1200.0 1204.0 1208.0 1212.0 1216.0 1220.0 1224.0 1228.0 1232.0 1236.0 1240.0 1244.0 1248.0 1252.0 1256.0 1260.0 1264.0 1268.0 1272.0 1276.0 1280.0 1284.0 1288.0 1292.0 1296.0 1300.0 1304.0 1308.0 1312.0 1316.0 1320.0 1324.0 1328.0 1332.0 1336.0 1340.0 1344.0 1348.0 1352.0 1356.0 1360.0 1364.0 1368.0 1372.0 1376.0 1380.0 1384.0 1388.0 1392.0 1396.0 1400.0 1404.0 1408.0 1412.0 1416.0 1420.0 1424.0 1428.0 1432.0 1436.0 1440.0 1444.0 1448.0 1452.0 1456.0 1460.0 1464.0 1468.0 1472.0 1476.0 1480.0 1484.0 1488.0 1492.0 1496.0 1500.0 1504.0 1508.0 1512.0 1516.0 1520.0 1524.0 1528.0 1532.0 1536.0 1540.0 1544.0 1548.0 1552.0 1556.0 1560.0 1564.0 1568.0 1572.0 1576.0 1580.0 1584.0 1588.0 1592.0 1596.0 1600.0 1604.0 1608.0 1612.0 1616.0 1620.0 1624.0 1628.0 1632.0 1636.0 1640.0 1644.0 1648.0 1652.0 1656.0 1660.0 1664.0 1668.0 1672.0 1676.0 1680.0 1684.0 1688.0 1692.0 1696.0 1700.0 1704.0 1708.0 1712.0 1716.0 1720.0 1724.0 1728.0 1732.0 1736.0 1740.0 1744.0 1748.0 1752.0 1756.0 1760.0 1764.0 1768.0 1772.0 1776.0 1780.0 1784.0 1788.0 1792.0 1796.0 1800.0 1804.0 1808.0 1812.0 1816.0 1820.0 1824.0 1828.0 1832.0 1836.0 1840.0 1844.0 1848.0 1852.0 1856.0 1860.0 1864.0 1868.0 1872.0 1876.0 1880.0 1884.0 1888.0 1892.0 1896.0 1900.0"
+        output_values="-5.035627186666667 -4.9577605600000005 -4.9214732 -4.84436256 -4.79446744 -4.7445723200000005 -4.68 -4.57674328 -4.46334528 -4.40437832 -4.34994728 -4.22747744 -4.15943864 -4.11861536 -4.018825120000002 -3.95532224 -3.88728344 -3.8101727999999997 -3.7103825600000007 -3.66048744 -3.55616128 -3.47905064 -3.3565808 -3.2885419999999996 -3.16153624 -3.12524888 -3.00277904 -2.94381208 -2.87123736 -2.77598304 -2.73515976 -2.67165688 -2.6036180799999995 -2.54465112 -2.49929192 -2.43578904 -2.4040376 -2.3133192000000005 -2.26342408 -2.1999212000000004 -2.14095424 -2.1092028 -2.0411639999999998 -1.96858928 -1.91415824 -1.85519128 -1.79622432 -1.72818552 -1.6737544800000002 -1.6374671200000002 -1.58303608 -1.5195332000000001 -1.4741739999999999 -1.4106711200000002 -1.3743837600000002 -1.3244886400000002 -1.2700576 -1.2201624800000002 -1.17026736 -1.1067644800000005 -1.0659412 -1.0205819999999999 -0.98883056 -0.94347136 -0.907184 -0.8754325599999999 -0.83007336 -0.78017824 -0.75296272 -0.71667536 -0.68945984 -0.6577084 -0.6304928799999999 -0.5896696 -0.5579181599999999 -0.53070264 -0.50348712 -0.47173568 -0.44452016 -0.41276872 -0.38555320000000004 -0.35833767999999994 -0.32205032 -0.2948348 -0.26308336 -0.23586784 -0.2041164 -0.17236496 -0.14514943999999996 -0.12246984 -0.09071839999999999 -0.07257472 -0.05443104 -0.03628736 0.0 0.0 0.0 0.0 0.0 0.0 0.0 0.0 0.0 0.0 0.0 0.0 0.0 0.0 0.05896696 0.08618248 0.11339799999999997 0.14968536000000002 0.18143679999999998 0.21318824 0.2494756 0.28576296 0.32205032 0.3628736 0.39008912 0.42637648 0.46719976 0.4989511999999999 0.5352385599999999 0.57152592 0.6078132799999999 0.63956472 0.66224432 0.69853168 0.7393549599999999 0.78017824 0.8164656 0.8618248 0.88904032 0.93439952 0.9752228000000001 1.0205819999999999 1.06140528 1.1203722399999998 1.17026736 1.22016248 1.27912944 1.31088088 1.37891968 1.43788664 1.52860504 1.5830360799999998 1.64200304 1.73725736 1.8007602399999998 1.84611944 1.91869416 1.98219704 2.06837952 2.11827464 2.1999212000000004 2.24981632 2.32692696 2.43578904 2.52197152 2.6081540000000003 2.66258504 2.76237528 2.82587816 2.90752472 2.9937072 3.05721008 3.13432072 3.2205032000000005 3.27947016 3.3565807999999997 3.44276328 3.54708944 3.6423437600000006 3.72399032 3.84646016 3.96439408 4.10047168 4.209333760000002 4.32726768 4.422522 4.5540636800000005 4.6992131200000005 4.82168296 4.93054504 5.02126344 5.143733280000001 5.20270024 5.39320888 5.520214640000002 5.62000488 5.710723280000002 5.81504944 5.92844744 6.059989120000001 6.128027920000001 6.25503368 6.36389576 6.45915008 6.554404400000001 6.6224432 6.72223344"/>
+      <!-- </xacro:if> -->
     </xacro:generic_thruster_macro>
     <!-- <xacro:thruster_module_first_order_basic_fcn_macro
