Commit message: Added some rviz stuff

File: simulation/mantaray_description/robots/rviz_robot.xacro (robot description, xacro)
@@ -32,5 +32,3 @@
     </gazebo>
   </xacro:mantaray_base>
-  <!-- Joint state publisher plugin -->
-  <xacro:default_joint_state_publisher namespace="$(arg namespace)" update_rate="10"/>
 </robot>

File: simulation/mantaray_description/urdf/base.xacro (robot description, xacro)
@@ -25,7 +25,8 @@
   <xacro:property name="visual_mesh_file" value="file://$(find mantaray_description)/meshes/visual_base_link.stl"/>
   <!-- Vehicle macro -->
-  <xacro:macro name="mantaray_base" params="namespace *gazebo">
+  <xacro:macro name="mantaray_base" params="namespace *gazebo use_simplified_mesh inertial_reference_frame">
       <!-- Rigid body description of the base link -->
       <link name="${namespace}/base_link">
+        <parent link="world"/>
         <!--
           Be careful to setup the coefficients for the inertial tensor,

File: simulation/mantaray_description/urdf/sensors.xacro (robot description, xacro)
@@ -16,7 +16,10 @@
   </xacro:default_pressure> -->
   <!-- IMU  -->
-  <xacro:default_imu namespace="${namespace}" parent_link="${namespace}/base_link">
+  <xacro:default_imu_macro
+    namespace="${namespace}"
+    parent_link="${namespace}/base_link"
+    inertial_reference_frame="${inertial_reference_frame}">
     <origin xyz="0 0 0" rpy="0 0 0"/>
-  </xacro:default_imu>
+  </xacro:default_imu_macro>
   <!-- Mount a camera  -->
   <!-- <xacro:default_camera namespace="${namespace}" parent_link="${namespace}/base_link" suffix="">
